Commit message: reduced mesh

File: roboy_xylophone/model.urdf (robot description, URDF)
Before this commit: robot roboy_xylophone, 22 links, 21 joints
Links:
- link base: geometry collision mesh filename=package://robots/roboy_xylophone/meshes/CAD/base.stl scale=0.001 0.001 0.001; visual mesh filename=package://robots/roboy_xylophone/meshes/CAD/base.stl scale=0.001 0.001 0.001
- link lower_arm_left: geometry collision mesh filename=package://robots/roboy_xylophone/meshes/CAD/lower_arm_left.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 scale=0.001 0.001 0.001; visual mesh filename=package://robots/roboy_xylophone/meshes/CAD/lower_arm_left.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 scale=0.001 0.001 0.001
- link torso: geometry collision mesh filename=package://robots/roboy_xylophone/meshes/CAD/torso.stl scale=0.001 0.001 0.001; visual mesh filename=package://robots/roboy_xylophone/meshes/CAD/torso.stl scale=0.001 0.001 0.001
- link upper_arm_left: geometry collision mesh filename=package://robots/roboy_xylophone/meshes/CAD/upper_arm_left.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 scale=0.001 0.001 0.001; visual mesh filename=package://robots/roboy_xylophone/meshes/CAD/upper_arm_left.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 scale=0.001 0.001 0.001
