Commit message: with visuals folder

File: yatr/model.urdf (robot description, URDF)
Before this commit: robot yatr, 4 links, 3 joints
Links:
- link base: geometry collision mesh filename=package://robots/yatr/meshes/collisions/base.stl scale=0.001 0.001 0.001; visual mesh filename=package://robots/yatr/meshes/visuals/base.stl scale=0.001 0.001 0.001
- link link0: geometry collision mesh filename=package://robots/yatr/meshes/collisions/link0.stl scale=0.001 0.001 0.001; visual mesh filename=package://robots/yatr/meshes/visuals/link0.stl scale=0.001 0.001 0.001
- link link1: geometry collision mesh filename=package://robots/yatr/meshes/collisions/link1.stl scale=0.001 0.001 0.001; visual mesh filename=package://robots/yatr/meshes/visuals/link1.stl scale=0.001 0.001 0.001
- link link2: geometry collision mesh filename=package://robots/yatr/meshes/collisions/link2.stl scale=0.001 0.001 0.001; visual mesh filename=package://robots/yatr/meshes/visuals/link2.stl scale=0.001 0.001 0.001
