Commit message: correct joint names

File: msj_platform/model.urdf (robot description, URDF)
Before this commit: robot msj_platform, 4 links, 3 joints
Links:
- removed link shere_link2
- added link sphere_link2, mass 0.03134065921190476; collision mesh filename=package://roboy_models/msj_platform/meshes/CAD/sphere_link2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 scale=0.001 0.001 0.001; visual mesh filename=package://roboy_models/msj_platform/meshes/CAD/sphere_link2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 scale=0.001 0.001 0.001
Joints:
- joint sphere_axis1: child shere_link2 -> sphere_link2
- joint sphere_axis2: parent shere_link2 -> sphere_link2

Commit message: updated sdf

File: msj_platform/model.urdf (robot description, URDF)
Before this commit: robot msj_platform, 4 links, 3 joints
Links:
- link base: geometry collision mesh filename=package://robots/msj_platform/meshes/CAD/base.stl scale=0.001 0.001 0.001; visual mesh filename=package://robots/msj_platform/meshes/CAD/base.stl scale=0.001 0.001 0.001
- link sphere_link1: geometry collision mesh filename=package://robots/msj_platform/meshes/CAD/sphere_link1.stl scale=0.001 0.001 0.001; visual mesh filename=package://robots/msj_platform/meshes/CAD/sphere_link1.stl scale=0.001 0.001 0.001
- link sphere_link2: geometry collision mesh filename=package://robots/msj_platform/meshes/CAD/sphere_link2.stl scale=0.001 0.001 0.001; visual mesh filename=package://robots/msj_platform/meshes/CAD/sphere_link2.stl scale=0.001 0.001 0.001
- link top: geometry collision mesh filename=package://robots/msj_platform/meshes/CAD/top.stl scale=0.001 0.001 0.001; visual mesh filename=package://robots/msj_platform/meshes/CAD/top.stl scale=0.001 0.001 0.001
Joints:
- joint sphere_axis0: axis 1 0 0 -> 1  0  0; origin xyz=-0.00088 -0.00205  0.217 rpy=0 0 0 -> xyz=-0.00088 -0.00205  0.217 rpy=0  0  0
- joint sphere_axis1: axis 0 1 0 -> 0  1  0; origin xyz=0 0 0 rpy=0 0 0 -> xyz=0  0  0 rpy=0  0  0
- joint sphere_axis2: axis 0 0 1 -> 0  0  1; origin xyz=0 0 0 rpy=0 0 0 -> xyz=0  0  0 rpy=0  0  0

Commit message: with collision shapes

File: msj_platform/model.urdf (robot description, URDF)
Before this commit: robot msj_platform, 7 links, 6 joints
Links:
- link base: geometry collision mesh filename=package://robots/msj_platform/meshes/collisions/base.stl scale=0.001 0.001 0.001; visual mesh filename=package://robots/msj_platform/meshes/visuals/base.stl scale=0.001 0.001 0.001
- link sphere_link1: geometry collision mesh filename=package://robots/msj_platform/meshes/collisions/sphere_link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 scale=0.001 0.001 0.001; visual mesh filename=package://robots/msj_platform/meshes/visuals/sphere_link1.s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 scale=0.001 0.001 0.001
- link sphere_link2: geometry collision mesh filename=package://robots/msj_platform/meshes/collisions/sphere_link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 scale=0.001 0.001 0.001; visual mesh filename=package://robots/msj_platform/meshes/visuals/sphere_link2.s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 scale=0.001 0.001 0.001
- link tlv_0: geometry collision mesh filename=package://robots/msj_platform/meshes/collisions/tlv_0.stl scale=0.001 0.001 0.001; visual mesh filename=package://robots/msj_platform/meshes/visuals/tlv_0.stl scale=0.001 0.001 0.001
- link tlv_1: geometry collision mesh filename=package://robots/msj_platform/meshes/collisions/tlv_1.stl scale=0.001 0.001 0.001; visual mesh filename=package://robots/msj_platform/meshes/visuals/tlv_1.stl scale=0.001 0.001 0.001
- link tlv_2: geometry collision mesh filename=package://robots/msj_platform/meshes/collisions/tlv_2.stl scale=0.001 0.001 0.001; visual mesh filename=package://robots/msj_platform/meshes/visuals/tlv_2.stl scale=0.001 0.001 0.001
- link top: geometry collision mesh filename=package://robots/msj_platform/meshes/collisions/top.stl scale=0.001 0.001 0.001; visual mesh filename=package://robots/msj_platform/meshes/visuals/top.stl scale=0.001 0.001 0.001
Joints:
- joint sphere_axis0: axis 1 0 0 -> 1  0  0; origin xyz=0.00157 -0.00449  0.102 rpy=0 0 0 -> xyz=0.00157 -0.00449  0.102 rpy=0  0  0
- joint sphere_axis1: origin xyz=0 0 0 rpy=0 0 0 -> xyz=0  0  0 rpy=0  0  0
- joint sphere_axis2: axis 0 0 1 -> 0  0  1; origin xyz=0 0 0 rpy=0 0 0 -> xyz=0  0  0 rpy=0  0  0
- joint tlv_sensor_0: axis 0 0 0 -> 0  0  0; origin xyz=-0.00566  0.01698  0.09455 rpy=0 0 0 -> xyz=-0.00566  0.01698  0.09455 rpy=0  0  0; type revolute -> fixed
- joint tlv_sensor_1: axis 0 0 0 -> 0  0  0; origin xyz=0.01259 0.00116 0.08334 rpy=0 0 0 -> xyz=0.01259  0.00116  0.08334 rpy=0  0  0; type revolute -> fixed
- joint tlv_sensor_2: axis 0 0 0 -> 0  0  0; origin xyz=-0.0139   0.00098  0.08529 rpy=0 0 0 -> xyz=-0.0139   0.00098  0.08529 rpy=0  0  0; type revolute -> fixed

File: rikshaw/model.urdf (robot description, URDF)
Before this commit: robot rikshaw, 14 links, 13 joints
Links:
- link bike: geometry collision mesh filename=package://robots/rikshaw/meshes/collisions/bike.stl scale=0.001 0.001 0.001; visual mesh filename=package://robots/rikshaw/meshes/visuals/bike.stl scale=0.001 0.001 0.001
- link foot_left: geometry collision mesh filename=package://robots/rikshaw/meshes/collisions/foot_left.stl scale=0.001 0.001 0.001; visual mesh filename=package://robots/rikshaw/meshes/visuals/foot_left.stl scale=0.001 0.001 0.001
- link foot_right: geometry collision mesh filename=package://robots/rikshaw/meshes/collisions/foot_right.stl scale=0.001 0.001 0.001; visual mesh filename=package://robots/rikshaw/meshes/visuals/foot_right.stl scale=0.001 0.001 0.001
- link front_part: geometry collision mesh filename=package://robots/rikshaw/meshes/collisions/front_part.stl scale=0.001 0.001 0.001; visual mesh filename=package://robots/rikshaw/meshes/visuals/front_part.stl scale=0.001 0.001 0.001
- link kurbel: geometry collision mesh filename=package://robots/rikshaw/meshes/collisions/kurbel.stl scale=0.001 0.001 0.001; visual mesh filename=package://robots/rikshaw/meshes/visuals/kurbel.stl scale=0.001 0.001 0.001
- link left_wheel: geometry collision mesh filename=package://robots/rikshaw/meshes/collisions/left_wheel.stl scale=0.001 0.001 0.001; visual mesh filename=package://robots/rikshaw/meshes/visuals/left_wheel.stl scale=0.001 0.001 0.001
- link leg_left: geometry collision mesh filename=package://robots/rikshaw/meshes/collisions/leg_left.stl scale=0.001 0.001 0.001; visual mesh filename=package://robots/rikshaw/meshes/visuals/leg_left.stl scale=0.001 0.001 0.001
- link leg_right: geometry collision mesh filename=package://robots/rikshaw/meshes/collisions/leg_right.stl scale=0.001 0.001 0.001; visual mesh filename=package://robots/rikshaw/meshes/visuals/leg_right.stl scale=0.001 0.001 0.001
- link pedal_left: geometry collision mesh filename=package://robots/rikshaw/meshes/collisions/pedal_left.stl scale=0.001 0.001 0.001; visual mesh filename=package://robots/rikshaw/meshes/visuals/pedal_left.stl scale=0.001 0.001 0.001
- link pedal_right: geometry collision mesh filename=package://robots/rikshaw/meshes/collisions/pedal_right.stl scale=0.001 0.001 0.001; visual mesh filename=package://robots/rikshaw/meshes/visuals/pedal_right.stl scale=0.001 0.001 0.001
- link right_wheel: geometry collision mesh filename=package://robots/rikshaw/meshes/collisions/right_wheel.stl scale=0.001 0.001 0.001; visual mesh filename=package://robots/rikshaw/meshes/visuals/right_wheel.stl scale=0.001 0.001 0.001
- link thigh_left: geometry collision mesh filename=package://robots/rikshaw/meshes/collisions/thigh_left.stl scale=0.001 0.001 0.001; visual mesh filename=package://robots/rikshaw/meshes/visuals/thigh_left.stl scale=0.001 0.001 0.001
- link thigh_right: geometry collision mesh filename=package://robots/rikshaw/meshes/collisions/thigh_right.stl scale=0.001 0.001 0.001; visual mesh filename=package://robots/rikshaw/meshes/visuals/thigh_right.stl scale=0.001 0.001 0.001
- link wheel_back: geometry collision mesh filename=package://robots/rikshaw/meshes/collisions/wheel_back.stl scale=0.001 0.001 0.001; visual mesh filename=package://robots/rikshaw/meshes/visuals/wheel_back.stl scale=0.001 0.001 0.001

File: roboy_arcade_maschine/model.urdf (robot description, URDF)
Before this commit: robot roboy_arcade_maschine, 4 links, 3 joints
Links:
- link base: geometry collision mesh filename=package://robots/roboy_arcade_maschine/meshes/collisions/ba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 scale=0.001 0.001 0.001; visual mesh filename=package://robots/roboy_arcade_maschine/meshes/visuals/base.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 scale=0.001 0.001 0.001
- link head: geometry collision mesh filename=package://robots/roboy_arcade_maschine/meshes/collisions/he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 scale=0.001 0.001 0.001; visual mesh filename=package://robots/roboy_arcade_maschine/meshes/visuals/head.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 scale=0.001 0.001 0.001
- link sphere_link1: geometry collision mesh filename=package://robots/roboy_arcade_maschine/meshes/collisions/sp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 scale=0.001 0.001 0.001; visual mesh filename=package://robots/roboy_arcade_maschine/meshes/visuals/spher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 scale=0.001 0.001 0.001
- link sphere_link2: geometry collision mesh filename=package://robots/roboy_arcade_maschine/meshes/collisions/sp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 scale=0.001 0.001 0.001; visual mesh filename=package://robots/roboy_arcade_maschine/meshes/visuals/spher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 scale=0.001 0.001 0.001
Joints:
- joint sphere_axis0: axis 1 0 0 -> 1  0  0; origin xyz=0.1525  0.19751 1.57964 rpy=0 0 0 -> xyz=0.1525   0.19751  1.57964 rpy=0  0  0
- joint sphere_axis1: origin xyz=0 0 0 rpy=0 0 0 -> xyz=0  0  0 rpy=0  0  0
- joint sphere_axis2: axis 0      0.17364 0.9848 -> 0       0.17364  0.9848; origin xyz=0 0 0 rpy=0 0 0 -> xyz=0  0  0 rpy=0  0  0

File: roboy_xylophone/model.urdf (robot description, URDF)
Before this commit: robot roboy_xylophone, 24 links, 23 joints
Links:
- link base: geometry collision mesh filename=package://robots/roboy_xylophone/meshes/collisions/base.stl scale=0.001 0.001 0.001; visual mesh filename=package://robots/roboy_xylophone/meshes/visuals/base.stl scale=0.001 0.001 0.001
- link elbow_left: geometry collision mesh filename=package://robots/roboy_xylophone/meshes/collisions/elbow_le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 scale=0.001 0.001 0.001; visual mesh filename=package://robots/roboy_xylophone/meshes/visuals/elbow_left.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 scale=0.001 0.001 0.001
- link elbow_right: geometry collision mesh filename=package://robots/roboy_xylophone/meshes/collisions/elbow_ri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 scale=0.001 0.001 0.001; visual mesh filename=package://robots/roboy_xylophone/meshes/visuals/elbow_right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 scale=0.001 0.001 0.001
- link head: geometry collision mesh filename=package://robots/roboy_xylophone/meshes/collisions/head.stl scale=0.001 0.001 0.001; visual mesh filename=package://robots/roboy_xylophone/meshes/visuals/head.stl scale=0.001 0.001 0.001
- link left_hand: geometry collision mesh filename=package://robots/roboy_xylophone/meshes/collisions/left_han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 scale=0.001 0.001 0.001; visual mesh filename=package://robots/roboy_xylophone/meshes/visuals/left_hand.s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 scale=0.001 0.001 0.001
- link left_stick_tip: geometry collision mesh filename=package://robots/roboy_xylophone/meshes/collisions/left_sti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 scale=0.001 0.001 0.001; visual mesh filename=package://robots/roboy_xylophone/meshes/visuals/left_stick_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 scale=0.001 0.001 0.001
- link lower_arm_left: geometry collision mesh filename=package://robots/roboy_xylophone/meshes/collisions/lower_ar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 scale=0.001 0.001 0.001; visual mesh filename=package://robots/roboy_xylophone/meshes/visuals/lower_arm_l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 scale=0.001 0.001 0.001
- link lower_arm_right: geometry collision mesh filename=package://robots/roboy_xylophone/meshes/collisions/lower_ar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 scale=0.001 0.001 0.001; visual mesh filename=package://robots/roboy_xylophone/meshes/visuals/lower_arm_r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 scale=0.001 0.001 0.001
- link right_hand: geometry collision mesh filename=package://robots/roboy_xylophone/meshes/collisions/right_ha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 scale=0.001 0.001 0.001; visual mesh filename=package://robots/roboy_xylophone/meshes/visuals/right_hand.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 scale=0.001 0.001 0.001
- link right_stick_tip: geometry collision mesh filename=package://robots/roboy_xylophone/meshes/collisions/right_st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 scale=0.001 0.001 0.001; visual mesh filename=package://robots/roboy_xylophone/meshes/visuals/right_stick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 scale=0.001 0.001 0.001
- link shere_head_link2: geometry collision mesh filename=package://robots/roboy_xylophone/meshes/collisions/shere_he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 scale=0.001 0.001 0.001; visual mesh filename=package://robots/roboy_xylophone/meshes/visuals/shere_head_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 scale=0.001 0.001 0.001
- link sphere_head_link1: geometry collision mesh filename=package://robots/roboy_xylophone/meshes/collisions/sphere_h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 scale=0.001 0.001 0.001; visual mesh filename=package://robots/roboy_xylophone/meshes/visuals/sphere_head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 scale=0.001 0.001 0.001
- link sphere_left_link1: geometry collision mesh filename=package://robots/roboy_xylophone/meshes/collisions/sphere_l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 scale=0.001 0.001 0.001; visual mesh filename=package://robots/roboy_xylophone/meshes/visuals/sphere_left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 scale=0.001 0.001 0.001
- link sphere_left_link2: geometry collision mesh filename=package://robots/roboy_xylophone/meshes/collisions/sphere_l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 scale=0.001 0.001 0.001; visual mesh filename=package://robots/roboy_xylophone/meshes/visuals/sphere_left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 scale=0.001 0.001 0.001
- link sphere_right_link1: geometry collision mesh filename=package://robots/roboy_xylophone/meshes/collisions/sphere_r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 scale=0.001 0.001 0.001; visual mesh filename=package://robots/roboy_xylophone/meshes/visuals/sphere_righ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 scale=0.001 0.001 0.001
- link sphere_right_link2: geometry collision mesh filename=package://robots/roboy_xylophone/meshes/collisions/sphere_r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 scale=0.001 0.001 0.001; visual mesh filename=package://robots/roboy_xylophone/meshes/visuals/sphere_righ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 scale=0.001 0.001 0.001
- link torso: geometry collision mesh filename=package://robots/roboy_xylophone/meshes/collisions/torso.stl scale=0.001 0.001 0.001; visual mesh filename=package://robots/roboy_xylophone/meshes/visuals/torso.stl scale=0.001 0.001 0.001
- link upper_arm_left: geometry collision mesh filename=package://robots/roboy_xylophone/meshes/collisions/upper_ar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 scale=0.001 0.001 0.001; visual mesh filename=package://robots/roboy_xylophone/meshes/visuals/upper_arm_l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 scale=0.001 0.001 0.001
- link upper_arm_right: geometry collision mesh filename=package://robots/roboy_xylophone/meshes/collisions/upper_ar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 scale=0.001 0.001 0.001; visual mesh filename=package://robots/roboy_xylophone/meshes/visuals/upper_arm_r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 scale=0.001 0.001 0.001
- link wrist_left_1: geometry collision mesh filename=package://robots/roboy_xylophone/meshes/collisions/wrist_le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 scale=0.001 0.001 0.001; visual mesh filename=package://robots/roboy_xylophone/meshes/visuals/wrist_left_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 scale=0.001 0.001 0.001
- link wrist_right_1: geometry collision mesh filename=package://robots/roboy_xylophone/meshes/collisions/wrist_ri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 scale=0.001 0.001 0.001; visual mesh filename=package://robots/roboy_xylophone/meshes/visuals/wrist_right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 scale=0.001 0.001 0.001
- link zed_camera: geometry collision mesh filename=package://robots/roboy_xylophone/meshes/collisions/zed_came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 scale=0.001 0.001 0.001; visual mesh filename=package://robots/roboy_xylophone/meshes/visuals/zed_camera.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 scale=0.001 0.001 0.001
- link zed_camera_left_lense: geometry collision mesh filename=package://robots/roboy_xylophone/meshes/collisions/zed_came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 scale=0.001 0.001 0.001; visual mesh filename=package://robots/roboy_xylophone/meshes/visuals/zed_camera_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 scale=0.001 0.001 0.001
- link zed_camera_right_lense: geometry collision mesh filename=package://robots/roboy_xylophone/meshes/collisions/zed_came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 scale=0.001 0.001 0.001; visual mesh filename=package://robots/roboy_xylophone/meshes/visuals/zed_camera_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 scale=0.001 0.001 0.001
Joints:
- joint left_stick_tip_joint: type revolute -> fixed
- joint right_stick_tip_joint: type revolute -> fixed

Commit message: Change 'fixed' to 'revolute'

File: msj_platform/model.urdf (robot description, URDF)
Before this commit: robot msj_platform, 7 links, 6 joints
Joints:
- joint tlv_sensor_0: type fixed -> revolute
- joint tlv_sensor_1: type fixed -> revolute
- joint tlv_sensor_2: type fixed -> revolute
