Commit message: with endeffector

File: rikshaw/model.urdf (robot description, URDF)
Before this commit: robot , 9 links, 10 joints
Links:
- link foot_left: geometry collision mesh filename=package://robots/rikshaw/meshes/CAD/foot_left.stl scale=0.001 0.001 0.001; visual mesh filename=package://robots/rikshaw/meshes/CAD/foot_left.stl scale=0.001 0.001 0.001
- link foot_right: geometry collision mesh filename=package://robots/rikshaw/meshes/CAD/foot_right.stl scale=0.001 0.001 0.001; visual mesh filename=package://robots/rikshaw/meshes/CAD/foot_right.stl scale=0.001 0.001 0.001
- link hip_and_bike: geometry collision mesh filename=package://robots/rikshaw/meshes/CAD/hip_and_bike.stl scale=0.001 0.001 0.001; visual mesh filename=package://robots/rikshaw/meshes/CAD/hip_and_bike.stl scale=0.001 0.001 0.001
- link leg_left: geometry collision mesh filename=package://robots/rikshaw/meshes/CAD/leg_left.stl scale=0.001 0.001 0.001; visual mesh filename=package://robots/rikshaw/meshes/CAD/leg_left.stl scale=0.001 0.001 0.001
- link leg_right: geometry collision mesh filename=package://robots/rikshaw/meshes/CAD/leg_right.stl scale=0.001 0.001 0.001; visual mesh filename=package://robots/rikshaw/meshes/CAD/leg_right.stl scale=0.001 0.001 0.001
- link pedal_left: geometry collision mesh filename=package://robots/rikshaw/meshes/CAD/pedal_left.stl scale=0.001 0.001 0.001; visual mesh filename=package://robots/rikshaw/meshes/CAD/pedal_left.stl scale=0.001 0.001 0.001
- link pedal_right: geometry collision mesh filename=package://robots/rikshaw/meshes/CAD/pedal_right.stl scale=0.001 0.001 0.001; visual mesh filename=package://robots/rikshaw/meshes/CAD/pedal_right.stl scale=0.001 0.001 0.001
- link thigh_left: geometry collision mesh filename=package://robots/rikshaw/meshes/CAD/thigh_left.stl scale=0.001 0.001 0.001; visual mesh filename=package://robots/rikshaw/meshes/CAD/thigh_left.stl scale=0.001 0.001 0.001
- link thigh_right: geometry collision mesh filename=package://robots/rikshaw/meshes/CAD/thigh_right.stl scale=0.001 0.001 0.001; visual mesh filename=package://robots/rikshaw/meshes/CAD/thigh_right.stl scale=0.001 0.001 0.001
Joints:
- joint joint_bike_left: origin xyz=8.92735  0.04379  0.07853 rpy=0  0  0 -> xyz=8.92735 0.04379 0.07853 rpy=0 0 0
- joint joint_bike_right: origin xyz=8.88816  0.12525 -0.1941 rpy=0  0  0 -> xyz=8.88816  0.12525 -0.1941 rpy=0 0 0
- joint joint_foot_left: origin xyz=-0.07933 -0.60427 -0.02402 rpy=0  0  0 -> xyz=-0.07933 -0.60427 -0.02402 rpy=0 0 0
- joint joint_foot_right: axis 0  0  1 -> 0 0 1; origin xyz=0.19902 -0.52452  0.01406 rpy=0  0  0 -> xyz=0.19902 -0.52452  0.01406 rpy=0 0 0
- joint joint_hip_left: axis 0  0  1 -> 0 0 1; origin xyz=9.186    1.11463  0.3261 rpy=0  0  0 -> xyz=9.186   1.11463 0.3261 rpy=0 0 0
- joint joint_hip_right: axis 0  0  1 -> 0 0 1; origin xyz=9.07449  1.20389 -0.4342 rpy=0  0  0 -> xyz=9.07449  1.20389 -0.4342 rpy=0 0 0
- joint joint_knee_left: axis 0  0  1 -> 0 0 1; origin xyz=0.01209 -0.65657 -0.02503 rpy=0  0  0 -> xyz=0.01209 -0.65657 -0.02503 rpy=0 0 0
- joint joint_knee_right: origin xyz=-0.43148 -0.25074 -0.00687 rpy=0  0  0 -> xyz=-0.43148 -0.25074 -0.00687 rpy=0 0 0
- joint joint_pedal_left: axis 0  0  1 -> 0 0 1; origin xyz=0.09815 -0.26057  0.26692 rpy=0  0  0 -> xyz=0.09815 -0.26057  0.26692 rpy=0 0 0
- joint joint_pedal_right: origin xyz=-0.15088  0.23913 -0.26828 rpy=0  0  0 -> xyz=-0.15088  0.23913 -0.26828 rpy=0 0 0

Commit message: with steering

File: rikshaw/model.urdf (robot description, URDF)
Before this commit: robot rikshaw, 37 links, 36 joints
Joints:
- joint joint_foot_left_tip: type fixed -> revolute
- joint joint_foot_right_tip: type fixed -> revolute
- joint zed_camera_left: type fixed -> revolute
- joint zed_camera_mount: type fixed -> revolute
- joint zed_camera_right: type fixed -> revolute

Commit message: Added joint limits

File: rikshaw/model.urdf (robot description, URDF)
Before this commit: robot rikshaw, 37 links, 36 joints
Joints:
- joint joint_foot_left: limit lower=-3.14159265359 upper=3.14159265359 effort=0.0 velocity=0.0 -> lower=-0.2 upper=0.2 effort=0.0 velocity=0.0
- joint joint_foot_right: limit lower=-3.14159265359 upper=3.14159265359 effort=0.0 velocity=0.0 -> lower=-0.2 upper=0.2 effort=0.0 velocity=0.0
- joint joint_hip_left: limit lower=-3.14159265359 upper=3.14159265359 effort=0.0 velocity=0.0 -> lower=-0.3 upper=1.5 effort=0.0 velocity=0.0
- joint joint_hip_right: limit lower=-3.14159265359 upper=3.14159265359 effort=0.0 velocity=0.0 -> lower=-1.5 upper=0.3 effort=0.0 velocity=0.0
- joint joint_knee_left: limit lower=-3.14159265359 upper=3.14159265359 effort=0.0 velocity=0.0 -> lower=0.0 upper=1.5 effort=0.0 velocity=0.0
- joint joint_knee_right: limit lower=-3.14159265359 upper=3.14159265359 effort=0.0 velocity=0.0 -> lower=-1.5 upper=0.0 effort=0.0 velocity=0.0

Commit message: renamed tes_robot

File: rikshaw/model.urdf (robot description, URDF)
Before this commit: robot rikshaw, 37 links, 36 joints
Joints:
- joint joint_foot_left: limit lower=-0.2 upper=0.2 effort=0.0 velocity=0.0 -> lower=-0.5 upper=0.5 effort=0.0 velocity=0.0
- joint joint_foot_right: limit lower=-0.2 upper=0.2 effort=0.0 velocity=0.0 -> lower=-0.5 upper=0.5 effort=0.0 velocity=0.0
- joint joint_hip_left: limit lower=-0.3 upper=1.5 effort=0.0 velocity=0.0 -> lower=-1.5 upper=1.5 effort=0.0 velocity=0.0
- joint joint_hip_right: limit lower=-1.5 upper=0.3 effort=0.0 velocity=0.0 -> lower=-1.5 upper=1.5 effort=0.0 velocity=0.0

Commit message: changed joint limits

File: rikshaw/model.urdf (robot description, URDF)
Before this commit: robot rikshaw, 37 links, 36 joints
Joints:
- joint joint_foot_left: limit lower=-3.14159265359 upper=3.14159265359 effort=0.0 velocity=0.0 -> lower=-0.6 upper=0.6 effort=0.0 velocity=0.0
- joint joint_foot_right: limit lower=-3.14159265359 upper=3.14159265359 effort=0.0 velocity=0.0 -> lower=-0.6 upper=0.6 effort=0.0 velocity=0.0
- joint joint_hip_left: limit lower=-3.14159265359 upper=3.14159265359 effort=0.0 velocity=0.0 -> lower=-1.9 upper=0.4 effort=0.0 velocity=0.0
- joint joint_hip_right: limit lower=-3.14159265359 upper=3.14159265359 effort=0.0 velocity=0.0 -> lower=-1.9 upper=0.4 effort=0.0 velocity=0.0
- joint joint_knee_left: limit lower=-3.14159265359 upper=3.14159265359 effort=0.0 velocity=0.0 -> lower=0.0 upper=2.6 effort=0.0 velocity=0.0
- joint joint_knee_right: limit lower=-3.14159265359 upper=3.14159265359 effort=0.0 velocity=0.0 -> lower=-2.6 upper=0.0 effort=0.0 velocity=0.0

Commit message: Added joint limits

File: rikshaw/model.urdf (robot description, URDF)
Before this commit: robot rikshaw, 37 links, 36 joints
Joints:
- joint joint_foot_right: limit lower=-0.6 upper=0.6 effort=0.0 velocity=0.0 -> lower=-0.8 upper=0.8 effort=0.0 velocity=0.0
- joint joint_hip_right: limit lower=-1.9 upper=0.4 effort=0.0 velocity=0.0 -> lower=-3.14159265359 upper=3.14159265359 effort=0.0 velocity=0.0
- joint joint_knee_right: axis 0  1  0 -> 0  -1  0; limit lower=-2.6 upper=0.0 effort=0.0 velocity=0.0 -> lower=0.0 upper=3.14159265359 effort=0.0 velocity=0.0

Commit message: redid joint limits from Simon's push of new model

File: rikshaw/model.urdf (robot description, URDF)
Before this commit: robot rikshaw, 37 links, 36 joints
Joints:
- joint joint_foot_left: limit lower=-3.14159265359 upper=3.14159265359 effort=0.0 velocity=0.0 -> lower=-0.6 upper=0.6 effort=0.0 velocity=0.0
- joint joint_foot_right: limit lower=-3.14159265359 upper=3.14159265359 effort=0.0 velocity=0.0 -> lower=-0.6 upper=0.6 effort=0.0 velocity=0.0
- joint joint_hip_left: limit lower=-3.14159265359 upper=3.14159265359 effort=0.0 velocity=0.0 -> lower=-1.8 upper=0.4 effort=0.0 velocity=0.0
- joint joint_hip_right: limit lower=-3.14159265359 upper=3.14159265359 effort=0.0 velocity=0.0 -> lower=-1.8 upper=0.4 effort=0.0 velocity=0.0
- joint joint_knee_left: limit lower=-3.14159265359 upper=3.14159265359 effort=0.0 velocity=0.0 -> lower=0.0 upper=2.0 effort=0.0 velocity=0.0
- joint joint_knee_right: limit lower=-3.14159265359 upper=3.14159265359 effort=0.0 velocity=0.0 -> lower=-2.0 upper=0.0 effort=0.0 velocity=0.0
