Commit message: New rikshaw

File: rikshaw/model.urdf (robot description, URDF)
Before this commit: robot rikshaw, 67 links, 66 joints
Links:
- removed link rikshaw__bike
- removed link rikshaw__foot_left
- removed link rikshaw__foot_left_tip
- removed link rikshaw__foot_right
- removed link rikshaw__foot_right_tip
- removed link rikshaw__front_part
- removed link rikshaw__head
- removed link rikshaw__index_left_link0
- removed link rikshaw__index_left_link1
- removed link rikshaw__index_left_link2
- removed link rikshaw__index_right_link0
- removed link rikshaw__index_right_link1
- removed link rikshaw__index_right_link2
- removed link rikshaw__kurbel
- removed link rikshaw__left_shoulder_link1
- removed link rikshaw__left_shoulder_link2
- removed link rikshaw__left_wheel
- removed link rikshaw__leg_left
- removed link rikshaw__leg_right
- removed link rikshaw__little_left_link0
- removed link rikshaw__little_left_link1
- removed link rikshaw__little_left_link2
- removed link rikshaw__little_right_link0
- removed link rikshaw__little_right_link1
- removed link rikshaw__little_right_link2
- removed link rikshaw__lower_arm_left
- removed link rikshaw__lower_arm_right
- removed link rikshaw__middle_left_link0
- removed link rikshaw__middle_left_link1
- removed link rikshaw__middle_left_link2
- removed link rikshaw__middle_right_link0
- removed link rikshaw__middle_right_link1
- removed link rikshaw__middle_right_link2
- removed link rikshaw__palm_left
- removed link rikshaw__palm_right
- removed link rikshaw__pedal_left
- removed link rikshaw__pedal_right
- removed link rikshaw__right_shoulder_link1
- removed link rikshaw__right_shoulder_link2
- removed link rikshaw__right_wheel
- removed link rikshaw__ring_left_link0
- removed link rikshaw__ring_left_link1
- removed link rikshaw__ring_left_link2
- removed link rikshaw__ring_right_link0
- removed link rikshaw__ring_right_link1
- removed link rikshaw__ring_right_link2
- removed link rikshaw__sphere_head_link1
- removed link rikshaw__sphere_head_link2
- removed link rikshaw__thigh_left
- removed link rikshaw__thigh_right
- removed link rikshaw__thumb_left_link0
- removed link rikshaw__thumb_left_link1
- removed link rikshaw__thumb_left_link2
- removed link rikshaw__thumb_right_link0
- removed link rikshaw__thumb_right_link1
- removed link rikshaw__thumb_right_link2
- removed link rikshaw__torso
- removed link rikshaw__upper_arm_left
- removed link rikshaw__upper_arm_right
- removed link rikshaw__wheel_back
- removed link rikshaw__wrist_left_sphere_link1
- removed link rikshaw__wrist_left_sphere_link2
- removed link rikshaw__wrist_right_sphere_link1
- removed link rikshaw__wrist_right_sphere_link2
- removed link rikshaw__zed_camera
- removed link rikshaw__zed_camera_left_lense
- removed link rikshaw__zed_camera_right_lense
- added link bike, mass 21.819480362884757; collision mesh filename=package://robots/rikshaw/meshes/collisions/bike.stl scale=0.001 0.001 0.001; visual mesh filename=package://robots/rikshaw/meshes/visuals/bike.stl scale=0.001 0.001 0.001
- added link foot_left, mass 0.7293868680453512; collision mesh filename=package://robots/rikshaw/meshes/collisions/foot_left.stl scale=0.001 0.001 0.001; visual mesh filename=package://robots/rikshaw/meshes/visuals/foot_left.stl scale=0.001 0.001 0.001
- added link foot_left_tip, mass 0.27793994464342403; collision mesh filename=package://robots/rikshaw/meshes/collisions/foot_left_tip.stl scale=0.001 0.001 0.001; visual mesh filename=package://robots/rikshaw/meshes/visuals/foot_left_tip.stl scale=0.001 0.001 0.001
- added link foot_right, mass 0.729389451072159; collision mesh filename=package://robots/rikshaw/meshes/collisions/foot_right.stl scale=0.001 0.001 0.001; visual mesh filename=package://robots/rikshaw/meshes/visuals/foot_right.stl scale=0.001 0.001 0.001
- added link foot_right_tip, mass 0.27795073699830286; collision mesh filename=package://robots/rikshaw/meshes/collisions/foot_right_tip.s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 scale=0.001 0.001 0.001; visual mesh filename=package://robots/rikshaw/meshes/visuals/foot_right_tip.stl scale=0.001 0.001 0.001
- added link front_part, mass 16.81067246564987; collision mesh filename=package://robots/rikshaw/meshes/collisions/front_part.stl scale=0.001 0.001 0.001; visual mesh filename=package://robots/rikshaw/meshes/visuals/front_part.stl scale=0.001 0.001 0.001
- added link head, mass 2.118808936153909; collision mesh filename=package://robots/rikshaw/meshes/collisions/head.stl scale=0.001 0.001 0.001; visual mesh filename=package://robots/rikshaw/meshes/visuals/head.stl scale=0.001 0.001 0.001
- added link index_left_link0, mass 0.01078315363645507; collision mesh filename=package://robots/rikshaw/meshes/collisions/index_left_link0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 scale=0.001 0.001 0.001; visual mesh filename=package://robots/rikshaw/meshes/visuals/index_left_link0.stl scale=0.001 0.001 0.001
- added link index_left_link1, mass 0.008727346342048834; collision mesh filename=package://robots/rikshaw/meshes/collisions/index_left_link1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 scale=0.001 0.001 0.001; visual mesh filename=package://robots/rikshaw/meshes/visuals/index_left_link1.stl scale=0.001 0.001 0.001
- added link index_left_link2, mass 0.007230503768900909; collision mesh filename=package://robots/rikshaw/meshes/collisions/index_left_link2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 scale=0.001 0.001 0.001; visual mesh filename=package://robots/rikshaw/meshes/visuals/index_left_link2.stl scale=0.001 0.001 0.001
- added link index_right_link0, mass 0.010783226463222334; collision mesh filename=package://robots/rikshaw/meshes/collisions/index_right_link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 scale=0.001 0.001 0.001; visual mesh filename=package://robots/rikshaw/meshes/visuals/index_right_link0.s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 scale=0.001 0.001 0.001
- added link index_right_link1, mass 0.008727441849375963; collision mesh filename=package://robots/rikshaw/meshes/collisions/index_right_link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 scale=0.001 0.001 0.001; visual mesh filename=package://robots/rikshaw/meshes/visuals/index_right_link1.s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 scale=0.001 0.001 0.001
- added link index_right_link2, mass 0.007230613589821098; collision mesh filename=package://robots/rikshaw/meshes/collisions/index_right_link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 scale=0.001 0.001 0.001; visual mesh filename=package://robots/rikshaw/meshes/visuals/index_right_link2.s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 scale=0.001 0.001 0.001
- added link kurbel, mass 2.7832708381108002; collision mesh filename=package://robots/rikshaw/meshes/collisions/kurbel.stl scale=0.001 0.001 0.001; visual mesh filename=package://robots/rikshaw/meshes/visuals/kurbel.stl scale=0.001 0.001 0.001
- added link left_shoulder_link1, mass 0.046754318188270985; collision mesh filename=package://robots/rikshaw/meshes/collisions/left_shoulder_li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 scale=0.001 0.001 0.001; visual mesh filename=package://robots/rikshaw/meshes/visuals/left_shoulder_link1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 scale=0.001 0.001 0.001
- added link left_shoulder_link2, mass 0.031341649376529494; collision mesh filename=package://robots/rikshaw/meshes/collisions/left_shoulder_li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 scale=0.001 0.001 0.001; visual mesh filename=package://robots/rikshaw/meshes/visuals/left_shoulder_link2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 scale=0.001 0.001 0.001
- added link left_wheel, mass 13.340163929097853; collision mesh filename=package://robots/rikshaw/meshes/collisions/left_wheel.stl scale=0.001 0.001 0.001; visual mesh filename=package://robots/rikshaw/meshes/visuals/left_wheel.stl scale=0.001 0.001 0.001
- added link leg_left, mass 5.742617323881256; collision mesh filename=package://robots/rikshaw/meshes/collisions/leg_left.stl scale=0.001 0.001 0.001; visual mesh filename=package://robots/rikshaw/meshes/visuals/leg_left.stl scale=0.001 0.001 0.001
- added link leg_right, mass 5.741522183296095; collision mesh filename=package://robots/rikshaw/meshes/collisions/leg_right.stl scale=0.001 0.001 0.001; visual mesh filename=package://robots/rikshaw/meshes/visuals/leg_right.stl scale=0.001 0.001 0.001
- added link little_left_link0, mass 0.010783173954625098; collision mesh filename=package://robots/rikshaw/meshes/collisions/little_left_link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 scale=0.001 0.001 0.001; visual mesh filename=package://robots/rikshaw/meshes/visuals/little_left_link0.s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 scale=0.001 0.001 0.001
- added link little_left_link1, mass 0.008727381894054248; collision mesh filename=package://robots/rikshaw/meshes/collisions/little_left_link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 scale=0.001 0.001 0.001; visual mesh filename=package://robots/rikshaw/meshes/visuals/little_left_link1.s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 scale=0.001 0.001 0.001
- added link little_left_link2, mass 0.007230544692585402; collision mesh filename=package://robots/rikshaw/meshes/collisions/little_left_link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 scale=0.001 0.001 0.001; visual mesh filename=package://robots/rikshaw/meshes/visuals/little_left_link2.s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 scale=0.001 0.001 0.001
- added link little_right_link0, mass 0.010783208913438909; collision mesh filename=package://robots/rikshaw/meshes/collisions/little_right_lin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 scale=0.001 0.001 0.001; visual mesh filename=package://robots/rikshaw/meshes/visuals/little_right_link0.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 scale=0.001 0.001 0.001
- added link little_right_link1, mass 0.008727399884658343; collision mesh filename=package://robots/rikshaw/meshes/collisions/little_right_lin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 scale=0.001 0.001 0.001; visual mesh filename=package://robots/rikshaw/meshes/visuals/little_right_link1.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 scale=0.001 0.001 0.001
- added link little_right_link2, mass 0.007230564904666386; collision mesh filename=package://robots/rikshaw/meshes/collisions/little_right_lin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 scale=0.001 0.001 0.001; visual mesh filename=package://robots/rikshaw/meshes/visuals/little_right_link2.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 scale=0.001 0.001 0.001
- added link lower_arm_left, mass 7.123102043007604; collision mesh filename=package://robots/rikshaw/meshes/collisions/lower_arm_left.s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 scale=0.001 0.001 0.001; visual mesh filename=package://robots/rikshaw/meshes/visuals/lower_arm_left.stl scale=0.001 0.001 0.001
- added link lower_arm_right, mass 7.123104239811117; collision mesh filename=package://robots/rikshaw/meshes/collisions/lower_arm_right.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 scale=0.001 0.001 0.001; visual mesh filename=package://robots/rikshaw/meshes/visuals/lower_arm_right.stl scale=0.001 0.001 0.001
- added link middle_left_link0, mass 0.010783098914055156; collision mesh filename=package://robots/rikshaw/meshes/collisions/middle_left_link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 scale=0.001 0.001 0.001; visual mesh filename=package://robots/rikshaw/meshes/visuals/middle_left_link0.s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 scale=0.001 0.001 0.001
- added link middle_left_link1, mass 0.008727362475596008; collision mesh filename=package://robots/rikshaw/meshes/collisions/middle_left_link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 scale=0.001 0.001 0.001; visual mesh filename=package://robots/rikshaw/meshes/visuals/middle_left_link1.s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 scale=0.001 0.001 0.001
- added link middle_left_link2, mass 0.007230534463346676; collision mesh filename=package://robots/rikshaw/meshes/collisions/middle_left_link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 scale=0.001 0.001 0.001; visual mesh filename=package://robots/rikshaw/meshes/visuals/middle_left_link2.s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 scale=0.001 0.001 0.001
- added link middle_right_link0, mass 0.010783222786021226; collision mesh filename=package://robots/rikshaw/meshes/collisions/middle_right_lin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 scale=0.001 0.001 0.001; visual mesh filename=package://robots/rikshaw/meshes/visuals/middle_right_link0.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 scale=0.001 0.001 0.001
- added link middle_right_link1, mass 0.008727454453508098; collision mesh filename=package://robots/rikshaw/meshes/collisions/middle_right_lin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 scale=0.001 0.001 0.001; visual mesh filename=package://robots/rikshaw/meshes/visuals/middle_right_link1.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 scale=0.001 0.001 0.001
- added link middle_right_link2, mass 0.007230650401745365; collision mesh filename=package://robots/rikshaw/meshes/collisions/middle_right_lin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 scale=0.001 0.001 0.001; visual mesh filename=package://robots/rikshaw/meshes/visuals/middle_right_link2.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 scale=0.001 0.001 0.001
- added link palm_left, mass 0.4014213812126051; collision mesh filename=package://robots/rikshaw/meshes/collisions/palm_left.stl scale=0.001 0.001 0.001; visual mesh filename=package://robots/rikshaw/meshes/visuals/palm_left.stl scale=0.001 0.001 0.001
- added link palm_right, mass 0.41273188866593385; collision mesh filename=package://robots/rikshaw/meshes/collisions/palm_right.stl scale=0.001 0.001 0.001; visual mesh filename=package://robots/rikshaw/meshes/visuals/palm_right.stl scale=0.001 0.001 0.001
- added link pedal_left, mass 0.9460025886020074; collision mesh filename=package://robots/rikshaw/meshes/collisions/pedal_left.stl scale=0.001 0.001 0.001; visual mesh filename=package://robots/rikshaw/meshes/visuals/pedal_left.stl scale=0.001 0.001 0.001
- added link pedal_right, mass 0.946002588602011; collision mesh filename=package://robots/rikshaw/meshes/collisions/pedal_right.stl scale=0.001 0.001 0.001; visual mesh filename=package://robots/rikshaw/meshes/visuals/pedal_right.stl scale=0.001 0.001 0.001
- added link right_shoulder_link1, mass 0.046737542469703665; collision mesh filename=package://robots/rikshaw/meshes/collisions/right_shoulder_l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 scale=0.001 0.001 0.001; visual mesh filename=package://robots/rikshaw/meshes/visuals/right_shoulder_link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 scale=0.001 0.001 0.001
- added link right_shoulder_link2, mass 0.03133944344667861; collision mesh filename=package://robots/rikshaw/meshes/collisions/right_shoulder_l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 scale=0.001 0.001 0.001; visual mesh filename=package://robots/rikshaw/meshes/visuals/right_shoulder_link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 scale=0.001 0.001 0.001
- added link right_wheel, mass 13.340163929097852; collision mesh filename=package://robots/rikshaw/meshes/collisions/right_wheel.stl scale=0.001 0.001 0.001; visual mesh filename=package://robots/rikshaw/meshes/visuals/right_wheel.stl scale=0.001 0.001 0.001
- added link ring_left_link0, mass 0.01078319636299043; collision mesh filename=package://robots/rikshaw/meshes/collisions/ring_left_link0.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 scale=0.001 0.001 0.001; visual mesh filename=package://robots/rikshaw/meshes/visuals/ring_left_link0.stl scale=0.001 0.001 0.001
- added link ring_left_link1, mass 0.008727381460149852; collision mesh filename=package://robots/rikshaw/meshes/collisions/ring_left_link1.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 scale=0.001 0.001 0.001; visual mesh filename=package://robots/rikshaw/meshes/visuals/ring_left_link1.stl scale=0.001 0.001 0.001
- added link ring_left_link2, mass 0.007230598064083806; collision mesh filename=package://robots/rikshaw/meshes/collisions/ring_left_link2.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 scale=0.001 0.001 0.001; visual mesh filename=package://robots/rikshaw/meshes/visuals/ring_left_link2.stl scale=0.001 0.001 0.001
- added link ring_right_link0, mass 0.010783248840452798; collision mesh filename=package://robots/rikshaw/meshes/collisions/ring_right_link0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 scale=0.001 0.001 0.001; visual mesh filename=package://robots/rikshaw/meshes/visuals/ring_right_link0.stl scale=0.001 0.001 0.001
- added link ring_right_link1, mass 0.00872746416092259; collision mesh filename=package://robots/rikshaw/meshes/collisions/ring_right_link1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 scale=0.001 0.001 0.001; visual mesh filename=package://robots/rikshaw/meshes/visuals/ring_right_link1.stl scale=0.001 0.001 0.001
- added link ring_right_link2, mass 0.007230552864674504; collision mesh filename=package://robots/rikshaw/meshes/collisions/ring_right_link2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 scale=0.001 0.001 0.001; visual mesh filename=package://robots/rikshaw/meshes/visuals/ring_right_link2.stl scale=0.001 0.001 0.001
- added link sphere_head_link1, mass 0.017037660152065294; collision mesh filename=package://robots/rikshaw/meshes/collisions/sphere_head_link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 scale=0.001 0.001 0.001; visual mesh filename=package://robots/rikshaw/meshes/visuals/sphere_head_link1.s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 scale=0.001 0.001 0.001
- added link sphere_head_link2, mass 0.011421516918761764; collision mesh filename=package://robots/rikshaw/meshes/collisions/sphere_head_link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 scale=0.001 0.001 0.001; visual mesh filename=package://robots/rikshaw/meshes/visuals/sphere_head_link2.s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 scale=0.001 0.001 0.001
- added link thigh_left, mass 5.56358907681273; collision mesh filename=package://robots/rikshaw/meshes/collisions/thigh_left.stl scale=0.001 0.001 0.001; visual mesh filename=package://robots/rikshaw/meshes/visuals/thigh_left.stl scale=0.001 0.001 0.001
- added link thigh_right, mass 5.563526842051083; collision mesh filename=package://robots/rikshaw/meshes/collisions/thigh_right.stl scale=0.001 0.001 0.001; visual mesh filename=package://robots/rikshaw/meshes/visuals/thigh_right.stl scale=0.001 0.001 0.001
- added link thumb_left_link0, mass 0.010783039116982735; collision mesh filename=package://robots/rikshaw/meshes/collisions/thumb_left_link0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 scale=0.001 0.001 0.001; visual mesh filename=package://robots/rikshaw/meshes/visuals/thumb_left_link0.stl scale=0.001 0.001 0.001
- added link thumb_left_link1, mass 0.00872735081798693; collision mesh filename=package://robots/rikshaw/meshes/collisions/thumb_left_link1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 scale=0.001 0.001 0.001; visual mesh filename=package://robots/rikshaw/meshes/visuals/thumb_left_link1.stl scale=0.001 0.001 0.001
- added link thumb_left_link2, mass 0.00723049056417055; collision mesh filename=package://robots/rikshaw/meshes/collisions/thumb_left_link2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 scale=0.001 0.001 0.001; visual mesh filename=package://robots/rikshaw/meshes/visuals/thumb_left_link2.stl scale=0.001 0.001 0.001
- added link thumb_right_link0, mass 0.010783131534927236; collision mesh filename=package://robots/rikshaw/meshes/collisions/thumb_right_link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 scale=0.001 0.001 0.001; visual mesh filename=package://robots/rikshaw/meshes/visuals/thumb_right_link0.s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 scale=0.001 0.001 0.001
- added link thumb_right_link1, mass 0.008726839160214994; collision mesh filename=package://robots/rikshaw/meshes/collisions/thumb_right_link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 scale=0.001 0.001 0.001; visual mesh filename=package://robots/rikshaw/meshes/visuals/thumb_right_link1.s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 scale=0.001 0.001 0.001
- added link thumb_right_link2, mass 0.007230558586521256; collision mesh filename=package://robots/rikshaw/meshes/collisions/thumb_right_link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 scale=0.001 0.001 0.001; visual mesh filename=package://robots/rikshaw/meshes/visuals/thumb_right_link2.s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 scale=0.001 0.001 0.001
- added link torso, mass 12.615235486751962; collision mesh filename=package://robots/rikshaw/meshes/collisions/torso.stl scale=0.001 0.001 0.001; visual mesh filename=package://robots/rikshaw/meshes/visuals/torso.stl scale=0.001 0.001 0.001
- added link upper_arm_left, mass 3.6086368702723797; collision mesh filename=package://robots/rikshaw/meshes/collisions/upper_arm_left.s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 scale=0.001 0.001 0.001; visual mesh filename=package://robots/rikshaw/meshes/visuals/upper_arm_left.stl scale=0.001 0.001 0.001
- added link upper_arm_right, mass 3.6087085067988065; collision mesh filename=package://robots/rikshaw/meshes/collisions/upper_arm_right.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 scale=0.001 0.001 0.001; visual mesh filename=package://robots/rikshaw/meshes/visuals/upper_arm_right.stl scale=0.001 0.001 0.001
- added link wheel_back, mass 13.340163929098475; collision mesh filename=package://robots/rikshaw/meshes/collisions/wheel_back.stl scale=0.001 0.001 0.001; visual mesh filename=package://robots/rikshaw/meshes/visuals/wheel_back.stl scale=0.001 0.001 0.001
- added link wrist_left_sphere_link1, mass 0.06978284193312742; collision mesh filename=package://robots/rikshaw/meshes/collisions/wrist_left_spher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 scale=0.001 0.001 0.001; visual mesh filename=package://robots/rikshaw/meshes/visuals/wrist_left_sphere_l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 scale=0.001 0.001 0.001
- added link wrist_left_sphere_link2, mass 0.04677754976643715; collision mesh filename=package://robots/rikshaw/meshes/collisions/wrist_left_spher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 scale=0.001 0.001 0.001; visual mesh filename=package://robots/rikshaw/meshes/visuals/wrist_left_sphere_l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 scale=0.001 0.001 0.001
- added link wrist_right_sphere_link1, mass 0.06978897865508384; collision mesh filename=package://robots/rikshaw/meshes/collisions/wrist_right_sphe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 scale=0.001 0.001 0.001; visual mesh filename=package://robots/rikshaw/meshes/visuals/wrist_right_sphere_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 scale=0.001 0.001 0.001
- added link wrist_right_sphere_link2, mass 0.0467775497412831; collision mesh filename=package://robots/rikshaw/meshes/collisions/wrist_right_sphe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 scale=0.001 0.001 0.001; visual mesh filename=package://robots/rikshaw/meshes/visuals/wrist_right_sphere_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 scale=0.001 0.001 0.001
- added link zed_camera, mass 0.009633907998289063; collision mesh filename=package://robots/rikshaw/meshes/collisions/zed_camera.stl scale=0.001 0.001 0.001; visual mesh filename=package://robots/rikshaw/meshes/visuals/zed_camera.stl scale=0.001 0.001 0.001
- added link zed_camera_left_lense, mass 0.005755421853194515; collision mesh filename=package://robots/rikshaw/meshes/collisions/zed_camera_left_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 scale=0.001 0.001 0.001; visual mesh filename=package://robots/rikshaw/meshes/visuals/zed_camera_left_len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 scale=0.001 0.001 0.001
- added link zed_camera_right_lense, mass 0.0057554218519331405; collision mesh filename=package://robots/rikshaw/meshes/collisions/zed_camera_right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 scale=0.001 0.001 0.001; visual mesh filename=package://robots/rikshaw/meshes/visuals/zed_camera_right_le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 scale=0.001 0.001 0.001
Joints:
- removed joint rikshaw__elbow_left
- removed joint rikshaw__elbow_right
- removed joint rikshaw__index_left_joint0
- removed joint rikshaw__index_left_joint1
- removed joint rikshaw__index_left_joint2
- removed joint rikshaw__index_right_joint0
- removed joint rikshaw__index_right_joint1
- removed joint rikshaw__index_right_joint2
- removed joint rikshaw__joint_foot_left
- removed joint rikshaw__joint_foot_left_tip
- removed joint rikshaw__joint_foot_right
- removed joint rikshaw__joint_foot_right_tip
- removed joint rikshaw__joint_front
- removed joint rikshaw__joint_hip_left
- removed joint rikshaw__joint_hip_right
- removed joint rikshaw__joint_knee_left
- removed joint rikshaw__joint_knee_right
- removed joint rikshaw__joint_pedal
- removed joint rikshaw__joint_pedal_left
- removed joint rikshaw__joint_pedal_right
- removed joint rikshaw__joint_wheel_back
- removed joint rikshaw__joint_wheel_left
- removed joint rikshaw__joint_wheel_right
- removed joint rikshaw__left_shoulder_axis0
- removed joint rikshaw__left_shoulder_axis1
- removed joint rikshaw__left_shoulder_axis2
- removed joint rikshaw__little_left_joint0
- removed joint rikshaw__little_left_joint1
- removed joint rikshaw__little_left_joint2
- removed joint rikshaw__little_right_joint0
- removed joint rikshaw__little_right_joint1
- removed joint rikshaw__little_right_joint2
- removed joint rikshaw__middle_left_joint0
- removed joint rikshaw__middle_left_joint1
- removed joint rikshaw__middle_left_joint2
- removed joint rikshaw__middle_right_joint0
- removed joint rikshaw__middle_right_joint1
- removed joint rikshaw__middle_right_joint2
- removed joint rikshaw__right_shoulder_axis0
- removed joint rikshaw__right_shoulder_axis1
- removed joint rikshaw__right_shoulder_axis2
- removed joint rikshaw__ring_left_joint0
- removed joint rikshaw__ring_left_joint1
- removed joint rikshaw__ring_left_joint2
- removed joint rikshaw__ring_right_joint0
- removed joint rikshaw__ring_right_joint1
- removed joint rikshaw__ring_right_joint2
- removed joint rikshaw__sphere_head_axis0
- removed joint rikshaw__sphere_head_axis1
- removed joint rikshaw__sphere_head_axis2
- removed joint rikshaw__spine_joint
- removed joint rikshaw__thumb_left_joint0
- removed joint rikshaw__thumb_left_joint1
- removed joint rikshaw__thumb_left_joint2
- removed joint rikshaw__thumb_right_joint0
- removed joint rikshaw__thumb_right_joint1
- removed joint rikshaw__thumb_right_joint2
- removed joint rikshaw__wrist_left_sphere_axis0
- removed joint rikshaw__wrist_left_sphere_axis1
- removed joint rikshaw__wrist_left_sphere_axis2
- removed joint rikshaw__wrist_right_sphere_axis0
- removed joint rikshaw__wrist_right_sphere_axis1
- removed joint rikshaw__wrist_right_sphere_axis2
- removed joint rikshaw__zed_camera_left
- removed joint rikshaw__zed_camera_mount
- removed joint rikshaw__zed_camera_right
- added joint elbow_left: type revolute, parent upper_arm_left, child lower_arm_left, origin xyz=-0.00504 -0.23587 -0.18602 rpy=0 0 0, axis 0.03535 -0.65048  0.75869, limit lower=-1.2217304764 upper=0.0 effort=0.0 velocity=0.0
- added joint elbow_right: type revolute, parent upper_arm_right, child lower_arm_right, origin xyz=0.03327  0.2172  -0.2039 rpy=0 0 0, axis -0.03518 -0.64937 -0.75965, limit lower=-1.2217304764 upper=0.0 effort=0.0 velocity=0.0
- added joint index_left_joint0: type revolute, parent palm_left, child index_left_link0, origin xyz=0.04568 -0.20967 -0.18338 rpy=0 0 0, axis 0.99914  0.03916 -0.01297, limit lower=0.0 upper=0.0 effort=0.0 velocity=0.0
- added joint index_left_joint1: type revolute, parent index_left_link0, child index_left_link1, origin xyz=0.00103 -0.05003 -0.04297 rpy=0 0 0, axis 0.99914  0.03916 -0.01297, limit lower=0.0 upper=0.0 effort=0.0 velocity=0.0
- added joint index_left_joint2: type revolute, parent index_left_link1, child index_left_link2, origin xyz=-0.00231 -0.03944 -0.03332 rpy=0 0 0, axis 0.99914  0.03916 -0.01297, limit lower=0.0 upper=0.0 effort=0.0 velocity=0.0
- added joint index_right_joint0: type revolute, parent palm_right, child index_right_link0, origin xyz=-0.0529   0.12183 -0.1041 rpy=0 0 0, axis -0.96583 -0.17278  0.19313, limit lower=0.0 upper=0.0 effort=0.0 velocity=0.0
- added joint index_right_joint1: type revolute, parent index_right_link0, child index_right_link1, origin xyz=-0.00894  0.02577 -0.02168 rpy=0 0 0, axis -0.96583 -0.17278  0.19313, limit lower=0.0 upper=0.0 effort=0.0 velocity=0.0
- added joint index_right_joint2: type revolute, parent index_right_link1, child index_right_link2, origin xyz=-0.00658  0.02003 -0.01686 rpy=0 0 0, axis -0.96583 -0.17278  0.19313, limit lower=0.0 upper=0.0 effort=0.0 velocity=0.0
- added joint joint_foot_left: type revolute, parent leg_left, child foot_left, origin xyz=-0.00318  0.0135  -0.34912 rpy=0 0 0, axis 0 1 0, limit lower=-3.14159265359 upper=3.14159265359 effort=0.0 velocity=0.0
- added joint joint_foot_left_tip: type revolute, parent foot_left, child foot_left_tip, origin xyz=-0.06158 -0.024   -0.03743 rpy=0 0 0, axis 0 0 0, limit lower=0 upper=0 effort=0 velocity=0
- added joint joint_foot_right: type revolute, parent leg_right, child foot_right, origin xyz=0       0.0135  -0.34914 rpy=0 0 0, axis 0 1 0, limit lower=-3.14159265359 upper=3.14159265359 effort=0.0 velocity=0.0
- added joint joint_foot_right_tip: type revolute, parent foot_right, child foot_right_tip, origin xyz=-0.06197 -0.024   -0.03679 rpy=0 0 0, axis 0 0 0, limit lower=0 upper=0 effort=0 velocity=0
- added joint joint_front: type revolute, parent bike, child front_part, origin xyz=-0.94642  0       0.01116 rpy=0 0 0, axis 0 0 1, limit lower=-0.523598775598 upper=0.523598775598 effort=0.0 velocity=0.0
- added joint joint_hip_left: type revolute, parent bike, child thigh_left, origin xyz=0.2245  -0.20207  0.48902 rpy=0 0 0, axis 0 -1  0, limit lower=-3.14159265359 upper=3.14159265359 effort=0.0 velocity=0.0
- added joint joint_hip_right: type revolute, parent bike, child thigh_right, origin xyz=0.2245  0.16192 0.48902 rpy=0 0 0, axis 0 -1  0, limit lower=-3.14159265359 upper=3.14159265359 effort=0.0 velocity=0.0
- added joint joint_knee_left: type revolute, parent thigh_left, child leg_left, origin xyz=0.01653  0.02405 -0.30873 rpy=0 0 0, axis 0 -1  0, limit lower=-3.14159265359 upper=3.14159265359 effort=0.0 velocity=0.0
- added joint joint_knee_right: type revolute, parent thigh_right, child leg_right, origin xyz=0.01603  0.0077  -0.30874 rpy=0 0 0, axis 0 1 0, limit lower=-3.14159265359 upper=3.14159265359 effort=0.0 velocity=0.0
- added joint joint_pedal: type revolute, parent bike, child kurbel, origin xyz=0.0925  -0.035    0.00326 rpy=0 0 0, axis 0 1 0, limit lower=-3.14159265359 upper=3.14159265359 effort=0.0 velocity=0.0
- added joint joint_pedal_left: type revolute, parent kurbel, child pedal_left, origin xyz=0.01482 -0.15624 -0.16858 rpy=0 0 0, axis 0 -1  0, limit lower=-3.14159265359 upper=3.14159265359 effort=0.0 velocity=0.0
- added joint joint_pedal_right: type revolute, parent kurbel, child pedal_right, origin xyz=-0.01468  0.22498  0.16854 rpy=0 0 0, axis 0 1 0, limit lower=-3.14159265359 upper=3.14159265359 effort=0.0 velocity=0.0
- added joint joint_wheel_back: type revolute, parent bike, child wheel_back, origin xyz=0.53689 -0.06544  0.04941 rpy=0 0 0, axis 0 -1  0, limit lower=-3.14159265359 upper=3.14159265359 effort=0.0 velocity=0.0
- added joint joint_wheel_left: type revolute, parent front_part, child left_wheel, origin xyz=-0.052  -0.304   0.0345 rpy=0 0 0, axis 0 -1  0, limit lower=-3.14159265359 upper=3.14159265359 effort=0.0 velocity=0.0
- added joint joint_wheel_right: type revolute, parent front_part, child right_wheel, origin xyz=-0.052   0.338   0.0345 rpy=0 0 0, axis 0 1 0, limit lower=-3.14159265359 upper=3.14159265359 effort=0.0 velocity=0.0
- added joint left_shoulder_axis0: type revolute, parent torso, child left_shoulder_link1, origin xyz=0.01401 -0.29136  0.46864 rpy=0 0 0, axis 0.10384 -0.99454 -0.01031, limit lower=-3.14159265359 upper=3.14159265359 effort=0.0 velocity=0.0
- added joint left_shoulder_axis1: type revolute, parent left_shoulder_link1, child left_shoulder_link2, origin xyz=0 0 0 rpy=0 0 0, axis 0.98935  0.10435 -0.10145, limit lower=-3.14159265359 upper=3.14159265359 effort=0.0 velocity=0.0
- added joint left_shoulder_axis2: type revolute, parent left_shoulder_link2, child upper_arm_left, origin xyz=0 0 0 rpy=0 0 0, axis 0.01309 -0.75806 -0.65204, limit lower=-3.14159265359 upper=3.14159265359 effort=0.0 velocity=0.0
- added joint little_left_joint0: type revolute, parent palm_left, child little_left_link0, origin xyz=-0.30552  0.63249 -0.88201 rpy=0 0 0, axis 0.9663  -0.17142 -0.19199, limit lower=0.0 upper=0.0 effort=0.0 velocity=0.0
- added joint little_left_joint1: type revolute, parent little_left_link0, child little_left_link1, origin xyz=-0.00888 -0.02578 -0.02169 rpy=0 0 0, axis 0.9663  -0.17142 -0.19199, limit lower=0.0 upper=0.0 effort=0.0 velocity=0.0
- added joint little_left_joint2: type revolute, parent little_left_link1, child little_left_link2, origin xyz=-0.00723 -0.01991 -0.01673 rpy=0 0 0, axis 0.9663  -0.17142 -0.19199, limit lower=0.0 upper=0.0 effort=0.0 velocity=0.0
- added joint little_right_joint0: type revolute, parent palm_right, child little_right_link0, origin xyz=0.03566  0.11902 -0.10588 rpy=0 0 0, axis -0.99918  0.03777  0.01416, limit lower=0.0 upper=0.0 effort=0.0 velocity=0.0
- added joint little_right_joint1: type revolute, parent little_right_link0, child little_right_link1, origin xyz=0.00067  0.02643 -0.02269 rpy=0 0 0, axis -0.99918  0.03777  0.01416, limit lower=0.0 upper=0.0 effort=0.0 velocity=0.0
- added joint little_right_joint2: type revolute, parent little_right_link1, child little_right_link2, origin xyz=0.00088  0.02046 -0.01759 rpy=0 0 0, axis -0.99918  0.03777  0.01416, limit lower=0.0 upper=0.0 effort=0.0 velocity=0.0
- added joint middle_left_joint0: type revolute, parent palm_left, child middle_left_link0, origin xyz=-0.24936  0.62581 -0.89075 rpy=0 0 0, axis 0.9972  -0.02708 -0.06969, limit lower=0.0 upper=0.0 effort=0.0 velocity=0.0
- added joint middle_left_joint1: type revolute, parent middle_left_link0, child middle_left_link1, origin xyz=0.22525 -0.89746  0.65746 rpy=0 0 0, axis 0.9972  -0.02708 -0.06969, limit lower=0.0 upper=0.0 effort=0.0 velocity=0.0
- added joint middle_left_joint2: type revolute, parent middle_left_link1, child middle_left_link2, origin xyz=-0.22968  0.85052 -0.69749 rpy=0 0 0, axis 0.9972  -0.02708 -0.06969, limit lower=0.0 upper=0.0 effort=0.0 velocity=0.0
- added joint middle_right_joint0: type revolute, parent palm_right, child middle_right_link0, origin xyz=-0.02268  0.12501 -0.10823 rpy=0 0 0, axis -0.98992 -0.08135  0.11587, limit lower=0.0 upper=0.0 effort=0.0 velocity=0.0
- added joint middle_right_joint1: type revolute, parent middle_right_link0, child middle_right_link1, origin xyz=-0.00477  0.02631 -0.02233 rpy=0 0 0, axis -0.98992 -0.08135  0.11587, limit lower=0.0 upper=0.0 effort=0.0 velocity=0.0
- added joint middle_right_joint2: type revolute, parent middle_right_link1, child middle_right_link2, origin xyz=-0.00334  0.02041 -0.01735 rpy=0 0 0, axis -0.98992 -0.08135  0.11587, limit lower=0.0 upper=0.0 effort=0.0 velocity=0.0
- added joint right_shoulder_axis0: type revolute, parent torso, child right_shoulder_link1, origin xyz=-0.01699  0.29217  0.46803 rpy=0 0 0, axis 0.99999  0.00199 -0.00277, limit lower=-3.14159265359 upper=3.14159265359 effort=0.0 velocity=0.0
- added joint right_shoulder_axis1: type revolute, parent right_shoulder_link1, child right_shoulder_link2, origin xyz=0 0 0 rpy=0 0 0, axis 0.00079 0.65274 0.75757, limit lower=-3.14159265359 upper=3.14159265359 effort=0.0 velocity=0.0
- added joint right_shoulder_axis2: type revolute, parent right_shoulder_link2, child upper_arm_right, origin xyz=0 0 0 rpy=0 0 0, axis 0.11283  0.75267 -0.64864, limit lower=-3.14159265359 upper=3.14159265359 effort=0.0 velocity=0.0
- added joint ring_left_joint0: type revolute, parent palm_left, child ring_left_link0, origin xyz=-0.27576  0.62758 -0.8876 rpy=0 0 0, axis 0.99017 -0.07997 -0.1147, limit lower=0.0 upper=0.0 effort=0.0 velocity=0.0
- added joint ring_left_joint1: type revolute, parent ring_left_link0, child ring_left_link1, origin xyz=-0.00471 -0.02632 -0.02234 rpy=0 0 0, axis 0.99017 -0.07997 -0.1147, limit lower=0.0 upper=0.0 effort=0.0 velocity=0.0
- added joint ring_left_joint2: type revolute, parent ring_left_link1, child ring_left_link2, origin xyz=-0.004   -0.02036 -0.01727 rpy=0 0 0, axis 0.99017 -0.07997 -0.1147, limit lower=0.0 upper=0.0 effort=0.0 velocity=0.0
- added joint ring_right_joint0: type revolute, parent palm_right, child ring_right_link0, origin xyz=0.0037   0.12583 -0.11056 rpy=0 0 0, axis -0.99658 -0.03377  0.07539, limit lower=0.0 upper=0.0 effort=0.0 velocity=0.0
- added joint ring_right_joint1: type revolute, parent ring_right_link0, child ring_right_link1, origin xyz=-0.0026   0.02644 -0.02254 rpy=0 0 0, axis -0.99658 -0.03377  0.07539, limit lower=0.0 upper=0.0 effort=0.0 velocity=0.0
- added joint ring_right_joint2: type revolute, parent ring_right_link1, child ring_right_link2, origin xyz=-0.00165  0.02049 -0.01749 rpy=0 0 0, axis -0.99658 -0.03377  0.07539, limit lower=0.0 upper=0.0 effort=0.0 velocity=0.0
- added joint sphere_head_axis0: type revolute, parent torso, child sphere_head_link1, origin xyz=-0.01231  0       0.63022 rpy=0 0 0, axis -0.98394 -0.17741 -0.01922, limit lower=-0.523598775598 upper=0.523598775598 effort=0.0 velocity=0.0
- added joint sphere_head_axis1: type revolute, parent sphere_head_link1, child sphere_head_link2, origin xyz=0 0 0 rpy=0 0 0, axis -0.17738  0.98413 -0.00346, limit lower=-0.523598775598 upper=0.523598775598 effort=0.0 velocity=0.0
- added joint sphere_head_axis2: type revolute, parent sphere_head_link2, child head, origin xyz=0 0 0 rpy=0 0 0, axis -0.01953  0       0.9998, limit lower=-0.523598775598 upper=0.523598775598 effort=0.0 velocity=0.0
- added joint spine_joint: type revolute, parent bike, child torso, origin xyz=0.22048 -0.01442  0.69498 rpy=0 0 0, axis 0.01953  0      -0.9998, limit lower=-0.523598775598 upper=0.523598775598 effort=0.0 velocity=0.0
- added joint thumb_left_joint0: type revolute, parent palm_left, child thumb_left_link0, origin xyz=-0.0641  -0.00151 -0.12005 rpy=0 0 0, axis -0.93035 -0.29889 -0.21238, limit lower=0.0 upper=0.0 effort=0.0 velocity=0.0
- added joint thumb_left_joint1: type revolute, parent thumb_left_link0, child thumb_left_link1, origin xyz=0.02441 -0.04602 -0.04046 rpy=0 0 0, axis -0.93035 -0.29889 -0.21238, limit lower=0.0 upper=0.0 effort=0.0 velocity=0.0
- added joint thumb_left_joint2: type revolute, parent thumb_left_link1, child thumb_left_link2, origin xyz=0.02199 -0.03483 -0.0312 rpy=0 0 0, axis -0.93035 -0.29889 -0.21238, limit lower=0.0 upper=0.0 effort=0.0 velocity=0.0
- added joint thumb_right_joint0: type revolute, parent palm_right, child thumb_right_link0, origin xyz=-0.05052  0.02046 -0.07739 rpy=0 0 0, axis 0.93034 -0.29908  0.21216, limit lower=0.0 upper=0.0 effort=0.0 velocity=0.0
- added joint thumb_right_joint1: type revolute, parent thumb_right_link0, child thumb_right_link1, origin xyz=0.01271  0.02436 -0.02142 rpy=0 0 0, axis 0.93034 -0.29908  0.21216, limit lower=0.0 upper=0.0 effort=0.0 velocity=0.0
- added joint thumb_right_joint2: type revolute, parent thumb_right_link1, child thumb_right_link2, origin xyz=0.00951  0.01898 -0.01667 rpy=0 0 0, axis 0.93034 -0.29908  0.21216, limit lower=0.0 upper=0.0 effort=0.0 velocity=0.0
- added joint wrist_left_sphere_axis0: type revolute, parent lower_arm_left, child wrist_left_sphere_link1, origin xyz=0.2456  -0.87507  0.66462 rpy=0 0 0, axis -0.99869 -0.05101  0.0028, limit lower=-3.14159265359 upper=3.14159265359 effort=0.0 velocity=0.0
- added joint wrist_left_sphere_axis1: type revolute, parent wrist_left_sphere_link1, child wrist_left_sphere_link2, origin xyz=0 0 0 rpy=0 0 0, axis 0.03535 -0.65048  0.75869, limit lower=-3.14159265359 upper=3.14159265359 effort=0.0 velocity=0.0
- added joint wrist_left_sphere_axis2: type revolute, parent wrist_left_sphere_link2, child palm_left, origin xyz=-0.00322 -0.04271 -0.03955 rpy=0 0 0, axis 0.03688 -0.7578  -0.65143, limit lower=-3.14159265359 upper=3.14159265359 effort=0.0 velocity=0.0
- added joint wrist_right_sphere_axis0: type revolute, parent lower_arm_right, child wrist_right_sphere_link1, origin xyz=0.00171  0.18503 -0.14508 rpy=0 0 0, axis -0.99299  0.10853 -0.04678, limit lower=-3.14159265359 upper=3.14159265359 effort=0.0 velocity=0.0
- added joint wrist_right_sphere_axis1: type revolute, parent wrist_right_sphere_link1, child wrist_right_sphere_link2, origin xyz=0 0 0 rpy=0 0 0, axis -0.03535 -0.65048 -0.75869, limit lower=-3.14159265359 upper=3.14159265359 effort=0.0 velocity=0.0
- added joint wrist_right_sphere_axis2: type revolute, parent wrist_right_sphere_link2, child palm_right, origin xyz=0 0 0 rpy=0 0 0, axis 0.03688  0.7578  -0.65143, limit lower=-3.14159265359 upper=3.14159265359 effort=0.0 velocity=0.0
- added joint zed_camera_left: type revolute, parent zed_camera, child zed_camera_left_lense, origin xyz=-0.00138 -0.03848 -0.00785 rpy=0 0 0, axis 0 0 0, limit lower=0 upper=0 effort=0 velocity=0
- added joint zed_camera_mount: type revolute, parent head, child zed_camera, origin xyz=-0.06237 -0.02168  0.22039 rpy=0 0 0, axis 0 0 0, limit lower=0 upper=0 effort=0 velocity=0
- added joint zed_camera_right: type revolute, parent zed_camera, child zed_camera_right_lense, origin xyz=-0.00176  0.08149 -0.00786 rpy=0 0 0, axis 0 0 0, limit lower=0 upper=0 effort=0 velocity=0
