Commit message: Tried to pedal in simulation

File: rikshaw/model.urdf (robot description, URDF)
Before this commit: robot rikshaw, 67 links, 66 joints
Joints:
- joint wrist_left_sphere_axis0: limit lower=-3.14159265359 upper=3.14159265359 effort=0.0 velocity=0.0 -> lower=0 upper=0 effort=0.0 velocity=0.0
- joint wrist_right_sphere_axis0: limit lower=-3.14159265359 upper=3.14159265359 effort=0.0 velocity=0.0 -> lower=0 upper=0 effort=0.0 velocity=0.0

Commit message: Steering stuff

File: rikshaw/model.urdf (robot description, URDF)
Before this commit: robot rikshaw, 67 links, 66 joints
Joints:
- joint wrist_left_sphere_axis0: limit lower=0 upper=0 effort=0.0 velocity=0.0 -> lower=-3.14159265359 upper=3.14159265359 effort=0.0 velocity=0.0
- joint wrist_right_sphere_axis0: limit lower=0 upper=0 effort=0.0 velocity=0.0 -> lower=-3.14159265359 upper=3.14159265359 effort=0.0 velocity=0.0
