Commit message: renamed joint

File: human/model.urdf (robot description, URDF)
Before this commit: robot human, 62 links, 61 joints
Links:
- removed link 6dof_link1
- removed link 6dof_link2
- removed link 6dof_link3
- removed link 6dof_link4
- removed link 6dof_link5
- added link dof6_link1, mass 0.03806502884740436; collision mesh filename=package://robots/human/meshes/collisions/dof6_link1.stl scale=0.001 0.001 0.001; visual mesh filename=package://robots/human/meshes/visuals/dof6_link1.stl scale=0.001 0.001 0.001
- added link dof6_link2, mass 0.0029963725331776064; collision mesh filename=package://robots/human/meshes/collisions/dof6_link2.stl scale=0.001 0.001 0.001; visual mesh filename=package://robots/human/meshes/visuals/dof6_link2.stl scale=0.001 0.001 0.001
- added link dof6_link3, mass 0.015709236754408065; collision mesh filename=package://robots/human/meshes/collisions/dof6_link3.stl scale=0.001 0.001 0.001; visual mesh filename=package://robots/human/meshes/visuals/dof6_link3.stl scale=0.001 0.001 0.001
- added link dof6_link4, mass 0.029253556048299417; collision mesh filename=package://robots/human/meshes/collisions/dof6_link4.stl scale=0.001 0.001 0.001; visual mesh filename=package://robots/human/meshes/visuals/dof6_link4.stl scale=0.001 0.001 0.001
- added link dof6_link5, mass 0.029267161202751052; collision mesh filename=package://robots/human/meshes/collisions/dof6_link5.stl scale=0.001 0.001 0.001; visual mesh filename=package://robots/human/meshes/visuals/dof6_link5.stl scale=0.001 0.001 0.001
Joints:
- removed joint 6dof_axis0
- removed joint 6dof_axis1
- removed joint 6dof_axis2
- removed joint 6dof_axis3
- removed joint 6dof_axis4
- removed joint 6dof_axis5
- added joint dof6_axis0: type revolute, parent base, child dof6_link1, origin xyz=0.e+00 -1.e-05  1.e+00 rpy=0 0 0, axis 1 0 0, limit lower=-3.14159265359 upper=3.14159265359 effort=0.0 velocity=0.0
- added joint dof6_axis1: type revolute, parent dof6_link1, child dof6_link2, origin xyz=0 0 0 rpy=0 0 0, axis 0 1 0, limit lower=-3.14159265359 upper=3.14159265359 effort=0.0 velocity=0.0
- added joint dof6_axis2: type revolute, parent dof6_link2, child dof6_link3, origin xyz=0 0 0 rpy=0 0 0, axis 0 0 1, limit lower=-3.14159265359 upper=3.14159265359 effort=0.0 velocity=0.0
- added joint dof6_axis3: type prismatic, parent dof6_link3, child dof6_link4, origin xyz=0 0 0 rpy=0 0 0, axis -1  0  0, limit lower=-1.0 upper=1.0 effort=0.0 velocity=0.0
- added joint dof6_axis4: type prismatic, parent dof6_link4, child dof6_link5, origin xyz=0 0 0 rpy=0 0 0, axis 0 1 0, limit lower=-1.0 upper=1.0 effort=0.0 velocity=0.0
- added joint dof6_axis5: type prismatic, parent dof6_link5, child hip, origin xyz=0.e+00 1.e-05 0.e+00 rpy=0 0 0, axis 0 0 1, limit lower=-1.0 upper=1.0 effort=0.0 velocity=0.0
