Commit message: with manual joint axis

File: roboy_head/model.urdf (robot description, URDF)
Before this commit: robot roboy_head, 7 links, 6 joints
Joints:
- joint sphere_head_axis0: origin xyz=0       0       0.06647 rpy=0  0  0 -> xyz=0       0       0.06647 rpy=1  0  0
- joint sphere_head_axis1: axis -0.99215 -0.12498  0 -> 0 1 0
- joint sphere_head_axis2: limit lower=-0.523598775598 upper=0.523598775598 effort=0.0 velocity=0.0 -> lower=-1.5 upper=1.5 effort=0.0 velocity=0.0
- joint zed_camera_left: type fixed -> revolute
- joint zed_camera_mount: type fixed -> revolute
- joint zed_camera_right: type fixed -> revolute

Commit message: blabla

File: roboy_head/model.urdf (robot description, URDF)
Before this commit: robot roboy_head, 7 links, 6 joints
Joints:
- joint sphere_head_axis1: axis 0 1 0 -> 0 0 1
- joint sphere_head_axis2: axis 0  0  1 -> 0  1  0
