Commit message: cardsflow.urdf for CF, model.urdf for moveit

File: roboy_icecream/cardsflow.urdf (robot description, URDF)
Before this commit: robot roboy_icecream, 55 links, 54 joints
Links:
- removed link hand_left_index_link0
- removed link hand_left_index_link1
- removed link hand_left_index_link2
- removed link hand_left_little_link0
- removed link hand_left_little_link1
- removed link hand_left_little_link2
- removed link hand_left_middle_link0
- removed link hand_left_middle_link1
- removed link hand_left_middle_link2
- removed link hand_left_ring_link0
- removed link hand_left_ring_link1
- removed link hand_left_ring_link2
- removed link hand_left_thumb_link0
- removed link hand_left_thumb_link1
- removed link hand_left_thumb_link2
- removed link hand_right_index_link0
- removed link hand_right_index_link1
- removed link hand_right_index_link2
- removed link hand_right_little_link0
- removed link hand_right_little_link1
- removed link hand_right_little_link2
- removed link hand_right_middle_link0
- removed link hand_right_middle_link1
- removed link hand_right_middle_link2
- removed link hand_right_ring_link0
- removed link hand_right_ring_link1
- removed link hand_right_ring_link2
- removed link hand_right_thumb_link0
- removed link hand_right_thumb_link1
- removed link hand_right_thumb_link2
- removed link scooper
- removed link scooper_dummy_axis0
- removed link scooper_dummy_axis1
- removed link scooper_dummy_axis2
- removed link zed_camera
- removed link zed_camera_left_lense
- removed link zed_camera_right_lense
Joints:
- removed joint hand_left_index_joint0
- removed joint hand_left_index_joint1
- removed joint hand_left_index_joint2
- removed joint hand_left_little_joint0
- removed joint hand_left_little_joint1
- removed joint hand_left_little_joint2
- removed joint hand_left_middle_joint0
- removed joint hand_left_middle_joint1
- removed joint hand_left_middle_joint2
- removed joint hand_left_ring_joint0
- removed joint hand_left_ring_joint1
- removed joint hand_left_ring_joint2
- removed joint hand_left_thumb_joint0
- removed joint hand_left_thumb_joint1
- removed joint hand_left_thumb_joint2
- removed joint hand_right_index_joint0
- removed joint hand_right_index_joint1
- removed joint hand_right_index_joint2
- removed joint hand_right_little_joint0
- removed joint hand_right_little_joint1
- removed joint hand_right_little_joint2
- removed joint hand_right_middle_joint0
- removed joint hand_right_middle_joint1
- removed joint hand_right_middle_joint2
- removed joint hand_right_ring_joint0
- removed joint hand_right_ring_joint1
- removed joint hand_right_ring_joint2
- removed joint hand_right_thumb_joint0
- removed joint hand_right_thumb_joint1
- removed joint hand_right_thumb_joint2
- removed joint scooper_dummy_joint0
- removed joint scooper_dummy_joint1
- removed joint scooper_dummy_joint2
- removed joint scooper_palm
- removed joint zed_camera_left
- removed joint zed_camera_mount
- removed joint zed_camera_right
- joint shoulder_left_axis0: limit lower=-1.87 upper=0.88 effort=0.0 velocity=0.0 -> lower=-3.14159265359 upper=3.14159265359 effort=0.0 velocity=0.0
- joint shoulder_left_axis1: limit lower=-0.2 upper=1.463 effort=0.0 velocity=0.0 -> lower=-3.14159265359 upper=3.14159265359 effort=0.0 velocity=0.0
- joint shoulder_left_axis2: limit lower=-0.6 upper=0.6 effort=0.0 velocity=0.0 -> lower=-3.14159265359 upper=3.14159265359 effort=0.0 velocity=0.0
- joint shoulder_right_axis0: axis 1 0 0 -> 0.99863 -0.05074  0.01234; limit lower=-1.87 upper=0.88 effort=0.0 velocity=0.0 -> lower=-3.14 upper=3.14 effort=0.0 velocity=0.0
- joint shoulder_right_axis1: axis 0 1 0 -> -0.05101 -0.99844  0.02231; limit lower=-0.2 upper=1.463 effort=0.0 velocity=0.0 -> lower=-3.14 upper=3.14 effort=0.0 velocity=0.0
- joint shoulder_right_axis2: axis 0 0 1 -> 0.01118 -0.0229  -0.99967; limit lower=-0.6 upper=0.6 effort=0.0 velocity=0.0 -> lower=-3.14 upper=3.14 effort=0.0 velocity=0.0

Commit message: damn viapoints

File: roboy_icecream/cardsflow.urdf (robot description, URDF)
Before this commit: robot roboy_icecream, 18 links, 17 joints
Joints:
- joint shoulder_right_axis0: axis 0.99863 -0.05074  0.01234 -> 1 0 0
- joint shoulder_right_axis1: axis -0.05101 -0.99844  0.02231 -> 0 1 0
- joint shoulder_right_axis2: axis 0.01118 -0.0229  -0.99967 -> 0 0 1

Commit message: Remove icecream boxes

File: roboy_icecream/cardsflow.urdf (robot description, URDF)
Before this commit: robot roboy_icecream, 57 links, 56 joints
Links:
- removed link ice_left
- removed link ice_right
Joints:
- removed joint ice_tray_0
- removed joint ice_tray_1

File: roboy_icecream/model.urdf (robot description, URDF)
Before this commit: robot roboy_icecream, 22 links, 21 joints
Links:
- removed link ice_left
- removed link ice_right
Joints:
- removed joint ice_tray_0
- removed joint ice_tray_1

Commit message: left shoulder adapter, updated meshes in rviz

File: roboy_icecream/cardsflow.urdf (robot description, URDF)
Before this commit: robot roboy_icecream, 55 links, 54 joints
Links:
- removed link hand_left_index_link0
- removed link hand_left_index_link1
- removed link hand_left_index_link2
- removed link hand_left_little_link0
- removed link hand_left_little_link1
- removed link hand_left_little_link2
- removed link hand_left_middle_link0
- removed link hand_left_middle_link1
- removed link hand_left_middle_link2
- removed link hand_left_palm
- removed link hand_left_ring_link0
- removed link hand_left_ring_link1
- removed link hand_left_ring_link2
- removed link hand_left_thumb_link0
- removed link hand_left_thumb_link1
- removed link hand_left_thumb_link2
- removed link hand_right_index_link0
- removed link hand_right_index_link1
- removed link hand_right_index_link2
- removed link hand_right_little_link0
- removed link hand_right_little_link1
- removed link hand_right_little_link2
- removed link hand_right_middle_link0
- removed link hand_right_middle_link1
- removed link hand_right_middle_link2
- removed link hand_right_ring_link0
- removed link hand_right_ring_link1
- removed link hand_right_ring_link2
- removed link hand_right_thumb_link0
- removed link hand_right_thumb_link1
- removed link hand_right_thumb_link2
- removed link palm_right
- removed link scooper
- removed link scooper_target
- removed link sphere_link1
- removed link sphere_link2
- link arm_left_lower: mass 1.1243588187932434 -> 0.11243588187932435
- link arm_left_upper: mass 2.9509331504680603 -> 0.3010990375097506
- link arm_right_lower: mass 1.1302413328334573 -> 0.26996310025843295
- link arm_right_upper: mass 2.98314384024382 -> 0.30382570619625904
- link bike_back: mass 12.95134492036292 -> 1.2951344920362922
- link bike_front: mass 1286.0735575666731 -> 63.7307664696775
- link head: mass 2.049574035129589 -> 0.20495740351295888
- link neck_link1: mass 0.017038665636260372 -> 0.0017038665636260374
- link neck_link2: mass 0.011421521917888835 -> 0.0011421521917888836
- link pico_flexx: mass 0.015436810520105988 -> 0.0015436810520105988
- link shoulder_left_link1: mass 0.09036188404972216 -> 0.009036188404972216
- link shoulder_left_link2: mass 0.00711317010884494 -> 0.0007113170108844941
- link shoulder_right_link1: mass 0.09036760208789225 -> 0.009036760208789225
- link shoulder_right_link2: mass 0.007113171768782596 -> 0.0007113171768782597
- link torso: mass 11.519352383740124 -> 1.1519352383740125
- link zed_camera: mass 0.009633907989226701 -> 0.0009633907989226702
- link zed_camera_left_lense: mass 0.005755421856391891 -> 0.0005755421856391891
- link zed_camera_right_lense: mass 0.0057554218551259745 -> 0.0005755421855125974
- link zed_mini: mass 0.4361891515825777 -> 0.043618915158257776
Joints:
- removed joint hand_left_index_joint0
- removed joint hand_left_index_joint1
- removed joint hand_left_index_joint2
- removed joint hand_left_little_joint0
- removed joint hand_left_little_joint1
- removed joint hand_left_little_joint2
- removed joint hand_left_middle_joint0
- removed joint hand_left_middle_joint1
- removed joint hand_left_middle_joint2
- removed joint hand_left_ring_joint0
- removed joint hand_left_ring_joint1
- removed joint hand_left_ring_joint2
- removed joint hand_left_thumb_joint0
- removed joint hand_left_thumb_joint1
- removed joint hand_left_thumb_joint2
- removed joint hand_right_index_joint0
- removed joint hand_right_index_joint1
- removed joint hand_right_index_joint2
- removed joint hand_right_little_joint0
- removed joint hand_right_little_joint1
- removed joint hand_right_little_joint2
- removed joint hand_right_middle_joint0
- removed joint hand_right_middle_joint1
- removed joint hand_right_middle_joint2
- removed joint hand_right_ring_joint0
- removed joint hand_right_ring_joint1
- removed joint hand_right_ring_joint2
- removed joint hand_right_thumb_joint0
- removed joint hand_right_thumb_joint1
- removed joint hand_right_thumb_joint2
- removed joint palm_scooper
- removed joint scooper_target_axis0
- removed joint scooper_target_axis1
- removed joint scooper_target_axis2
- removed joint wrist_left
- removed joint wrist_right
- joint bike_steering: axis 0  0  1 -> 0 0 1; origin xyz=-0.00193 -1.20232 -0.903 rpy=0  0  0 -> xyz=-0.00193 -1.20232 -0.903 rpy=0 0 0
- joint elbow_left: limit lower=-3.14 upper=3.14 effort=0.0 velocity=0.0 -> lower=0.0 upper=0.0 effort=0.0 velocity=0.0; origin xyz=0.01342 -0.00741 -0.36229 rpy=0  0  0 -> xyz=0.01342 -0.00741 -0.36229 rpy=0 0 0
- joint elbow_right: limit lower=0.0 upper=10 effort=0.0 velocity=0.0 -> lower=0.0 upper=1.91986217719 effort=0.0 velocity=0.0; origin xyz=-0.013    0.00079 -0.3624 rpy=0  0  0 -> xyz=-0.013    0.00079 -0.3624 rpy=0 0 0
- joint neck_axis0: origin xyz=0       0.00152  0.71567 rpy=0  0  0 -> xyz=0      0.00152 0.71567 rpy=0 0 0
- joint neck_axis1: origin xyz=0  0  0 rpy=0  0  0 -> xyz=0 0 0 rpy=0 0 0
- joint neck_axis2: axis 0  0  1 -> 0 0 1; origin xyz=0  0  0 rpy=0  0  0 -> xyz=0 0 0 rpy=0 0 0
- joint shoulder_left_axis0: origin xyz=0.29189  0.01393  0.54489 rpy=0  0  0 -> xyz=0.29189 0.01393 0.54489 rpy=0 0 0
- joint shoulder_left_axis1: origin xyz=0  0  0 rpy=0  0  0 -> xyz=0 0 0 rpy=0 0 0
- joint shoulder_left_axis2: origin xyz=0  0  0 rpy=0  0  0 -> xyz=0 0 0 rpy=0 0 0
- joint shoulder_right_axis0: axis 1 0 0 -> 0.99863 -0.05074  0.01234; origin xyz=-0.29317  0.00923  0.5481 rpy=0  0  0 -> xyz=-0.29317  0.00923  0.5481 rpy=0 0 0
- joint shoulder_right_axis1: axis 0 1 0 -> -5.0740e-02 -9.9871e-01 -3.7000e-04; origin xyz=0  0  0 rpy=0  0  0 -> xyz=0 0 0 rpy=0 0 0
- joint shoulder_right_axis2: axis 0 0 1 -> 1.2340e-02 -2.5000e-04 -9.9992e-01; origin xyz=0  0  0 rpy=0  0  0 -> xyz=0 0 0 rpy=0 0 0
- joint spine: limit lower=-3.14 upper=3.14 effort=0.0 velocity=0.0 -> lower=0.0 upper=0.0 effort=0.0 velocity=0.0; origin xyz=0.00000000e+00  -2.00000000e-05   2.99330000e-01 rpy=0  0  0 -> xyz=0.0000e+00 -2.0000e-05  2.9933e-01 rpy=0 0 0
- joint zed_camera_left: axis 0  0  0 -> 0 0 0; origin xyz=0.03848 -0.00154 -0.00782 rpy=0  0  0 -> xyz=0.03848 -0.00154 -0.00782 rpy=0 0 0
- joint zed_camera_mount: axis 0  0  0 -> 0 0 0; origin xyz=0.02168 -0.05805  0.21956 rpy=0  0  0 -> xyz=0.02168 -0.05805  0.21956 rpy=0 0 0
- joint zed_camera_right: axis 0  0  0 -> 0 0 0; origin xyz=-0.08149 -0.00191 -0.00782 rpy=0  0  0 -> xyz=-0.08149 -0.00191 -0.00782 rpy=0 0 0
- joint zed_mini_attachement: axis 0  0  0 -> 0 0 0; origin xyz=0.00047 -0.10882  0.42356 rpy=0  0  0 -> xyz=0.00047 -0.10882  0.42356 rpy=0 0 0
- joint zed_pico_attachement: axis 0  0  0 -> 0 0 0; origin xyz=0.0576  -0.00665 -0.01668 rpy=0  0  0 -> xyz=0.0576  -0.00665 -0.01668 rpy=0 0 0

Commit message: with crossed tendons

File: roboy_icecream/cardsflow.urdf (robot description, URDF)
Before this commit: robot roboy_icecream, 19 links, 18 joints
Joints:
- joint shoulder_left_axis0: axis -0.99863 -0.05074  0.01234 -> 1 0 0
- joint shoulder_left_axis1: axis -0.05101  0.99844 -0.02231 -> 0 1 0
- joint shoulder_left_axis2: axis -0.01118 -0.0229  -0.99967 -> 0 0 1

File: roboy_icecream/model.urdf (robot description, URDF)
Before this commit: robot roboy_icecream, 20 links, 19 joints
Links:
- removed link hand_left_palm
- removed link palm_right
- removed link scooper
- removed link scooper_target
- removed link sphere_link1
- removed link sphere_link2
- added link pico_flexx, mass 0.0015436810520105988; collision mesh filename=package://robots/roboy_icecream/meshes/collisions/pico_flex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 scale=0.001 0.001 0.001; visual mesh filename=package://robots/roboy_icecream/meshes/visuals/pico_flexx.s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 scale=0.001 0.001 0.001
- added link zed_camera, mass 0.0009633907989226702; collision mesh filename=package://robots/roboy_icecream/meshes/collisions/zed_camer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 scale=0.001 0.001 0.001; visual mesh filename=package://robots/roboy_icecream/meshes/visuals/zed_camera.s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 scale=0.001 0.001 0.001
- added link zed_camera_left_lense, mass 0.0005755421856391891; collision mesh filename=package://robots/roboy_icecream/meshes/collisions/zed_camer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 scale=0.001 0.001 0.001; visual mesh filename=package://robots/roboy_icecream/meshes/visuals/zed_camera_l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 scale=0.001 0.001 0.001
- added link zed_camera_right_lense, mass 0.0005755421855125974; collision mesh filename=package://robots/roboy_icecream/meshes/collisions/zed_camer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 scale=0.001 0.001 0.001; visual mesh filename=package://robots/roboy_icecream/meshes/visuals/zed_camera_r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 scale=0.001 0.001 0.001
- added link zed_mini, mass 0.043618915158257776; collision mesh filename=package://robots/roboy_icecream/meshes/collisions/zed_mini.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 scale=0.001 0.001 0.001; visual mesh filename=package://robots/roboy_icecream/meshes/visuals/zed_mini.stl scale=0.001 0.001 0.001
- link arm_left_lower: mass 1.1243588187932434 -> 0.11243588187932435
- link arm_left_upper: mass 2.9509331504680603 -> 0.3010990375097506
- link arm_right_lower: mass 1.1302413328334573 -> 0.26996310025843295
- link arm_right_upper: mass 2.98314384024382 -> 0.30382570619625904
- link bike_back: mass 12.95134492036292 -> 1.2951344920362922
- link bike_front: mass 1286.0735575666731 -> 63.7307664696775
- link head: mass 2.049574035129589 -> 0.20495740351295888
- link neck_link1: mass 0.017038665636260372 -> 0.0017038665636260374
- link neck_link2: mass 0.011421521917888835 -> 0.0011421521917888836
- link shoulder_left_link1: mass 0.09036188404972216 -> 0.009036188404972216
- link shoulder_left_link2: mass 0.00711317010884494 -> 0.0007113170108844941
- link shoulder_right_link1: mass 0.09036760208789225 -> 0.009036760208789225
- link shoulder_right_link2: mass 0.007113171768782596 -> 0.0007113171768782597
- link torso: mass 11.519352383740124 -> 1.1519352383740125
Joints:
- removed joint palm_scooper
- removed joint scooper_target_axis0
- removed joint scooper_target_axis1
- removed joint scooper_target_axis2
- removed joint wrist_left
- removed joint wrist_right
- added joint zed_camera_left: type fixed, parent zed_camera, child zed_camera_left_lense, origin xyz=0.03848 -0.00154 -0.00782 rpy=0 0 0, axis 0 0 0, limit lower=0 upper=0 effort=0 velocity=0
- added joint zed_camera_mount: type fixed, parent head, child zed_camera, origin xyz=0.02168 -0.05805  0.21956 rpy=0 0 0, axis 0 0 0, limit lower=0 upper=0 effort=0 velocity=0
- added joint zed_camera_right: type fixed, parent zed_camera, child zed_camera_right_lense, origin xyz=-0.08149 -0.00191 -0.00782 rpy=0 0 0, axis 0 0 0, limit lower=0 upper=0 effort=0 velocity=0
- added joint zed_mini_attachement: type fixed, parent torso, child zed_mini, origin xyz=0.00047 -0.10882  0.42356 rpy=0 0 0, axis 0 0 0, limit lower=0 upper=0 effort=0 velocity=0
- added joint zed_pico_attachement: type fixed, parent zed_mini, child pico_flexx, origin xyz=0.0576  -0.00665 -0.01668 rpy=0 0 0, axis 0 0 0, limit lower=0 upper=0 effort=0 velocity=0
- joint bike_steering: axis 0  0  1 -> 0 0 1; origin xyz=-0.00193 -1.20232 -0.903 rpy=0  0  0 -> xyz=-0.00193 -1.20232 -0.903 rpy=0 0 0
- joint elbow_left: limit lower=-3.14 upper=3.14 effort=0.0 velocity=0.0 -> lower=0.0 upper=0.0 effort=0.0 velocity=0.0; origin xyz=0.01342 -0.00741 -0.36229 rpy=0  0  0 -> xyz=0.01342 -0.00741 -0.36229 rpy=0 0 0; type revolute -> fixed
- joint elbow_right: limit lower=0.0 upper=2.1 effort=0.0 velocity=0.0 -> lower=0.0 upper=1.91986217719 effort=0.0 velocity=0.0; origin xyz=-0.013    0.00079 -0.3624 rpy=0  0  0 -> xyz=-0.013    0.00079 -0.3624 rpy=0 0 0
- joint neck_axis0: origin xyz=0       0.00152  0.71567 rpy=0  0  0 -> xyz=0      0.00152 0.71567 rpy=0 0 0
- joint neck_axis1: origin xyz=0  0  0 rpy=0  0  0 -> xyz=0 0 0 rpy=0 0 0
- joint neck_axis2: axis 0  0  1 -> 0 0 1; origin xyz=0  0  0 rpy=0  0  0 -> xyz=0 0 0 rpy=0 0 0
- joint shoulder_left_axis0: origin xyz=0.29189  0.01393  0.54489 rpy=0  0  0 -> xyz=0.29189 0.01393 0.54489 rpy=0 0 0
- joint shoulder_left_axis1: origin xyz=0  0  0 rpy=0  0  0 -> xyz=0 0 0 rpy=0 0 0
- joint shoulder_left_axis2: origin xyz=0  0  0 rpy=0  0  0 -> xyz=0 0 0 rpy=0 0 0
- joint shoulder_right_axis0: axis 1 0 0 -> 0.99863 -0.05074  0.01234; limit lower=-1.57 upper=1.57 effort=0.0 velocity=0.0 -> lower=-3.14159265359 upper=3.14159265359 effort=0.0 velocity=0.0; origin xyz=-0.29317  0.00923  0.5481 rpy=0  0  0 -> xyz=-0.29317  0.00923  0.5481 rpy=0 0 0
- joint shoulder_right_axis1: axis 0 1 0 -> -5.0740e-02 -9.9871e-01 -3.7000e-04; limit lower=-0.2 upper=1.57 effort=0.0 velocity=0.0 -> lower=-3.14159265359 upper=3.14159265359 effort=0.0 velocity=0.0; origin xyz=0  0  0 rpy=0  0  0 -> xyz=0 0 0 rpy=0 0 0
- joint shoulder_right_axis2: axis 0 0 1 -> 1.2340e-02 -2.5000e-04 -9.9992e-01; limit lower=-0.3 upper=2.2 effort=0.0 velocity=0.0 -> lower=-3.14159265359 upper=3.14159265359 effort=0.0 velocity=0.0; origin xyz=0  0  0 rpy=0  0  0 -> xyz=0 0 0 rpy=0 0 0
- joint spine: limit lower=-3.14 upper=3.14 effort=0.0 velocity=0.0 -> lower=0.0 upper=0.0 effort=0.0 velocity=0.0; origin xyz=0.00000000e+00  -2.00000000e-05   2.99330000e-01 rpy=0  0  0 -> xyz=0.0000e+00 -2.0000e-05  2.9933e-01 rpy=0 0 0; type revolute -> fixed
