Commit message: Add rikshaw to icecream roboy

File: roboy_icecream/model.urdf (robot description, URDF)
Before this commit: robot roboy_icecream, 48 links, 47 joints
Links:
- added link bike, mass 21.819480362884757; collision mesh filename=package://robots/rikshaw/meshes/collisions/bike.stl scale=0.001 0.001 0.001; visual mesh filename=package://robots/rikshaw/meshes/visuals/bike.stl scale=0.001 0.001 0.001
- added link front_part, mass 16.81067246564987; collision mesh filename=package://robots/rikshaw/meshes/collisions/front_part.stl scale=0.001 0.001 0.001; visual mesh filename=package://robots/rikshaw/meshes/visuals/front_part.stl scale=0.001 0.001 0.001
- added link kurbel, mass 2.7832708381108002; collision mesh filename=package://robots/rikshaw/meshes/collisions/kurbel.stl scale=0.001 0.001 0.001; visual mesh filename=package://robots/rikshaw/meshes/visuals/kurbel.stl scale=0.001 0.001 0.001
- added link left_wheel, mass 13.340163929097853; collision mesh filename=package://robots/rikshaw/meshes/collisions/left_wheel.stl scale=0.001 0.001 0.001; visual mesh filename=package://robots/rikshaw/meshes/visuals/left_wheel.stl scale=0.001 0.001 0.001
- added link pedal_left, mass 0.9460025886020074; collision mesh filename=package://robots/rikshaw/meshes/collisions/pedal_left.stl scale=0.001 0.001 0.001; visual mesh filename=package://robots/rikshaw/meshes/visuals/pedal_left.stl scale=0.001 0.001 0.001
- added link pedal_right, mass 0.946002588602011; collision mesh filename=package://robots/rikshaw/meshes/collisions/pedal_right.stl scale=0.001 0.001 0.001; visual mesh filename=package://robots/rikshaw/meshes/visuals/pedal_right.stl scale=0.001 0.001 0.001
- added link right_wheel, mass 13.340163929097852; collision mesh filename=package://robots/rikshaw/meshes/collisions/right_wheel.stl scale=0.001 0.001 0.001; visual mesh filename=package://robots/rikshaw/meshes/visuals/right_wheel.stl scale=0.001 0.001 0.001
- added link wheel_back, mass 13.340163929098475; collision mesh filename=package://robots/rikshaw/meshes/collisions/wheel_back.stl scale=0.001 0.001 0.001; visual mesh filename=package://robots/rikshaw/meshes/visuals/wheel_back.stl scale=0.001 0.001 0.001
- added link world
Joints:
- added joint joint_front: type revolute, parent bike, child front_part, origin xyz=-0.94642  0       0.01116 rpy=0 0 0, axis 0 0 1, limit lower=-0.523598775598 upper=0.523598775598 effort=0.0 velocity=0.0
- added joint joint_pedal: type revolute, parent bike, child kurbel, origin xyz=0.0925  -0.035    0.00326 rpy=0 0 0, axis 0 1 0, limit lower=-3.14159265359 upper=3.14159265359 effort=0.0 velocity=0.0
- added joint joint_pedal_left: type revolute, parent kurbel, child pedal_left, origin xyz=0.01482 -0.15624 -0.16858 rpy=0 0 0, axis 0 -1  0, limit lower=-3.14159265359 upper=3.14159265359 effort=0.0 velocity=0.0
- added joint joint_pedal_right: type revolute, parent kurbel, child pedal_right, origin xyz=-0.01468  0.22498  0.16854 rpy=0 0 0, axis 0 1 0, limit lower=-3.14159265359 upper=3.14159265359 effort=0.0 velocity=0.0
- added joint joint_wheel_back: type revolute, parent bike, child wheel_back, origin xyz=0.53689 -0.06544  0.04941 rpy=0 0 0, axis 0 -1  0, limit lower=-3.14159265359 upper=3.14159265359 effort=0.0 velocity=0.0
- added joint joint_wheel_left: type revolute, parent front_part, child left_wheel, origin xyz=-0.052  -0.304   0.0345 rpy=0 0 0, axis 0 -1  0, limit lower=-3.14159265359 upper=3.14159265359 effort=0.0 velocity=0.0
- added joint joint_wheel_right: type revolute, parent front_part, child right_wheel, origin xyz=-0.052   0.338   0.0345 rpy=0 0 0, axis 0 1 0, limit lower=-3.14159265359 upper=3.14159265359 effort=0.0 velocity=0.0
- added joint spine_joint: type fixed, parent bike, child torso, origin xyz=0.22048 -0.01442  0.69498 rpy=0 0 0
- added joint world_joint: type fixed, parent world, child bike, origin xyz=0 0 0 rpy=0 0 0

Commit message: works for the arms

File: roboy_icecream/model.urdf (robot description, URDF)
Before this commit: robot roboy_icecream, 63 links, 62 joints
Joints:
- joint shoulder_left_axis0: axis -0.99863 -0.05074  0.01234 -> 1 0 0
- joint shoulder_left_axis1: axis -0.05101  0.99844 -0.02231 -> 0 1 0
- joint shoulder_left_axis2: axis -0.01118 -0.0229  -0.99967 -> 1 0 0
- joint shoulder_right_axis0: axis 0.99863 -0.05074  0.01234 -> 1 0 0
- joint shoulder_right_axis1: axis -0.05101 -0.99844  0.02231 -> 0 1 0
- joint shoulder_right_axis2: axis 0.01118 -0.0229  -0.99967 -> 1 0 0

Commit message: Revert "Add rikshaw to icecream roboy"
This reverts commit c7587a626199ba753bafb34015942056786c77d2.

File: roboy_icecream/model.urdf (robot description, URDF)
Before this commit: robot roboy_icecream, 57 links, 56 joints
Links:
- removed link bike
- removed link front_part
- removed link kurbel
- removed link left_wheel
- removed link pedal_left
- removed link pedal_right
- removed link right_wheel
- removed link wheel_back
- removed link world
Joints:
- removed joint joint_front
- removed joint joint_pedal
- removed joint joint_pedal_left
- removed joint joint_pedal_right
- removed joint joint_wheel_back
- removed joint joint_wheel_left
- removed joint joint_wheel_right
- removed joint spine_joint
- removed joint world_joint
