Commit message: add real sense, right shoulder

File: roboy_icecream/model.urdf (robot description, URDF)
Before this commit: robot roboy_icecream, 63 links, 62 joints
Links:
- removed link foot_left
- removed link foot_left_tip
- removed link foot_right
- removed link foot_right_tip
- removed link hip_left_tendon_guide
- removed link hip_right_tendon_guide
- removed link knee_left_tendon_guide
- removed link knee_right_tendon_guide
- removed link leg_left
- removed link leg_right
- removed link thigh_left
- removed link thigh_right
- removed link zed_camera
- removed link zed_camera_left_lense
- removed link zed_camera_right_lense
- added link bike, mass 21.819480362884757; collision mesh filename=package://robots/rikshaw/meshes/collisions/bike.stl scale=0.001 0.001 0.001; visual mesh filename=package://robots/rikshaw/meshes/visuals/bike.stl scale=0.001 0.001 0.001
- added link front_part, mass 16.81067246564987; collision mesh filename=package://robots/rikshaw/meshes/collisions/front_part.stl scale=0.001 0.001 0.001; visual mesh filename=package://robots/rikshaw/meshes/visuals/front_part.stl scale=0.001 0.001 0.001
- added link kurbel, mass 2.7832708381108002; collision mesh filename=package://robots/rikshaw/meshes/collisions/kurbel.stl scale=0.001 0.001 0.001; visual mesh filename=package://robots/rikshaw/meshes/visuals/kurbel.stl scale=0.001 0.001 0.001
- added link left_wheel, mass 13.340163929097853; collision mesh filename=package://robots/rikshaw/meshes/collisions/left_wheel.stl scale=0.001 0.001 0.001; visual mesh filename=package://robots/rikshaw/meshes/visuals/left_wheel.stl scale=0.001 0.001 0.001
- added link pedal_left, mass 0.9460025886020074; collision mesh filename=package://robots/rikshaw/meshes/collisions/pedal_left.stl scale=0.001 0.001 0.001; visual mesh filename=package://robots/rikshaw/meshes/visuals/pedal_left.stl scale=0.001 0.001 0.001
- added link pedal_right, mass 0.946002588602011; collision mesh filename=package://robots/rikshaw/meshes/collisions/pedal_right.stl scale=0.001 0.001 0.001; visual mesh filename=package://robots/rikshaw/meshes/visuals/pedal_right.stl scale=0.001 0.001 0.001
- added link real_sense_link, mass 0.00000171718499355
- added link right_wheel, mass 13.340163929097852; collision mesh filename=package://robots/rikshaw/meshes/collisions/right_wheel.stl scale=0.001 0.001 0.001; visual mesh filename=package://robots/rikshaw/meshes/visuals/right_wheel.stl scale=0.001 0.001 0.001
- added link wheel_back, mass 13.340163929098475; collision mesh filename=package://robots/rikshaw/meshes/collisions/wheel_back.stl scale=0.001 0.001 0.001; visual mesh filename=package://robots/rikshaw/meshes/visuals/wheel_back.stl scale=0.001 0.001 0.001
- added link world
- link arm_left_lower: mass 7.2740122404446215 -> 7.27401127870293
- link arm_left_palm: mass 0.8274415425908241 -> 0.8274404594388395
- link arm_left_upper: mass 3.6100762893022953 -> 3.6101133714243976
- link arm_right_lower: mass 7.274015985787583 -> 7.27400524780894
- link arm_right_palm: mass 0.8274574519860363 -> 0.8274696765002435
- link arm_right_upper: mass 3.61005569877743 -> 3.6102108682251886
- link hand_left_index_link0: mass 0.055846781261061205 -> 0.05584900095770278
- link hand_left_index_link1: mass 0.03081999399001323 -> 0.030810600216883144
- link hand_left_index_link2: mass 0.030336880161010958 -> 0.030337235888829715
- link hand_left_little_link0: mass 0.030820184437064607 -> 0.0308113741209532
- link hand_left_little_link1: mass 0.0308201844370646 -> 0.030811374120953198
- link hand_left_little_link2: mass 0.030336907136663423 -> 0.030336908642256268
- link hand_left_middle_link0: mass 0.0558465981006835 -> 0.055831334816546646
- link hand_left_middle_link1: mass 0.03082014849979441 -> 0.03081073881990825
- link hand_left_middle_link2: mass 0.030336901843144165 -> 0.03033633396737544
- link hand_left_ring_link0: mass 0.05584669978299005 -> 0.055852824780270094
- link hand_left_ring_link1: mass 0.03082008411770575 -> 0.030810597058291516
- link hand_left_ring_link2: mass 0.030336893727523316 -> 0.030336320395881453
- link hand_left_thumb_link0: mass 0.11643341043888081 -> 0.11643461952857805
- link hand_left_thumb_link1: mass 0.030820276240393865 -> 0.030824527684383127
- link hand_left_thumb_link2: mass 0.030336869955457046 -> 0.030335989064583388
- link hand_right_index_link0: mass 0.055845410084095805 -> 0.055849025991352386
- link hand_right_index_link1: mass 0.03082510142164794 -> 0.03081055844419456
- link hand_right_index_link2: mass 0.030337404031818088 -> 0.030337239357465594
- link hand_right_little_link0: mass 0.03082699976349422 -> 0.030813346429285876
- link hand_right_little_link1: mass 0.03082699976349423 -> 0.030813346429285935
- link hand_right_little_link2: mass 0.030337137210337213 -> 0.030337208280612718
- link hand_right_middle_link0: mass 0.055845163544770086 -> 0.05585161472558283
- link hand_right_middle_link1: mass 0.030825180144102245 -> 0.030811264606209175
- link hand_right_middle_link2: mass 0.03033726768863161 -> 0.030337290984439005
- link hand_right_ring_link0: mass 0.055843843204094676 -> 0.05584221000563185
- link hand_right_ring_link1: mass 0.030825311874925553 -> 0.03081221249464445
- link hand_right_ring_link2: mass 0.03033719311018232 -> 0.03033728342102297
- link hand_right_thumb_link0: mass 0.11642987827012777 -> 0.11643028119503748
- link hand_right_thumb_link1: mass 0.030824868780265316 -> 0.030826015044524206
- link hand_right_thumb_link2: mass 0.030336936473636927 -> 0.030336828875681794
- link head: mass 2.049574035129589 -> 2.049574035129534
- link neck_link1: mass 0.017038665636260372 -> 0.017038665636260365
- link shoulder_left_link1: mass 0.09036188404972213 -> 0.09036359201900478
- link shoulder_left_link2: mass 0.0071131701088449385 -> 0.007113170038864662
- link shoulder_right_link1: mass 0.09036491191489954 -> 0.0903636656787565
- link shoulder_right_link2: mass 0.00711317178967469 -> 0.007113171718499355
- link torso: mass 25.25525236846473 -> 11.588247145877938
- link wrist_left_link1: mass 0.09036188404972215 -> 0.09036359201900472
- link wrist_left_link2: mass 0.007113171769630984 -> 0.007113170038864663
- link wrist_right_link1: mass 0.09036361367400472 -> 0.09036366567875653
- link wrist_right_link2: mass 0.007113172058538673 -> 0.0071131715008991465
Joints:
- removed joint hip_left_axis0
- removed joint hip_left_axis1
- removed joint hip_right_axis0
- removed joint hip_right_axis1
- removed joint joint_foot_left
- removed joint joint_foot_left_tip
- removed joint joint_foot_right
- removed joint joint_foot_right_tip
- removed joint knee_left_axis0
- removed joint knee_left_axis1
- removed joint knee_right_axis0
- removed joint knee_right_axis1
- removed joint zed_camera_left
- removed joint zed_camera_mount
- removed joint zed_camera_right
- added joint joint_front: type revolute, parent bike, child front_part, origin xyz=-0.94642  0       0.01116 rpy=0 0 0, axis 0 0 1, limit lower=-0.523598775598 upper=0.523598775598 effort=0.0 velocity=0.0
- added joint joint_pedal: type revolute, parent bike, child kurbel, origin xyz=0.0925  -0.035    0.00326 rpy=0 0 0, axis 0 1 0, limit lower=-3.14159265359 upper=3.14159265359 effort=0.0 velocity=0.0
- added joint joint_pedal_left: type revolute, parent kurbel, child pedal_left, origin xyz=0.01482 -0.15624 -0.16858 rpy=0 0 0, axis 0 -1  0, limit lower=-3.14159265359 upper=3.14159265359 effort=0.0 velocity=0.0
- added joint joint_pedal_right: type revolute, parent kurbel, child pedal_right, origin xyz=-0.01468  0.22498  0.16854 rpy=0 0 0, axis 0 1 0, limit lower=-3.14159265359 upper=3.14159265359 effort=0.0 velocity=0.0
- added joint joint_wheel_back: type revolute, parent bike, child wheel_back, origin xyz=0.53689 -0.06544  0.04941 rpy=0 0 0, axis 0 -1  0, limit lower=-3.14159265359 upper=3.14159265359 effort=0.0 velocity=0.0
- added joint joint_wheel_left: type revolute, parent front_part, child left_wheel, origin xyz=-0.052  -0.304   0.0345 rpy=0 0 0, axis 0 -1  0, limit lower=-3.14159265359 upper=3.14159265359 effort=0.0 velocity=0.0
- added joint joint_wheel_right: type revolute, parent front_part, child right_wheel, origin xyz=-0.052   0.338   0.0345 rpy=0 0 0, axis 0 1 0, limit lower=-3.14159265359 upper=3.14159265359 effort=0.0 velocity=0.0
- added joint real_sense_joint: type fixed, parent shoulder_right_link1, child real_sense_link, origin xyz=-0.27306  0.01109  0.34684 rpy=0 0 0
- added joint spine_joint: type fixed, parent bike, child torso, origin xyz=0.22048 -0.01442  0.69498 rpy=0 0 -1.5708
- added joint world_joint: type fixed, parent world, child bike, origin xyz=0 0 0 rpy=0 0 0
- joint elbow_left: axis 0.99863  0.05074 -0.01234 -> 0.04893 -0.82665  0.56057; limit lower=0.0 upper=0.0 effort=0.0 velocity=0.0 -> lower=-3.14159265359 upper=3.14159265359 effort=0.0 velocity=0.0; origin xyz=0.00707 -0.00681 -0.30096 rpy=0  0  0 -> xyz=0.16849 -0.14194 -0.20242 rpy=0 0 0
- joint elbow_right: axis 0.99863 -0.05074  0.01234 -> 0.04893  0.82665 -0.56057; limit lower=0.0 upper=0.0 effort=0.0 velocity=0.0 -> lower=-3.14159265359 upper=3.14159265359 effort=0.0 velocity=0.0; origin xyz=-0.00816 -0.00684 -0.30497 rpy=0  0  0 -> xyz=-0.16894 -0.14055 -0.20436 rpy=0 0 0
- joint hand_left_index_joint0: axis -0.98736 -0.04706  0.15134 -> -0.12702  0.87986 -0.45793; limit lower=0.0 upper=0.0 effort=0.0 velocity=0.0 -> lower=-3.14159265359 upper=3.14159265359 effort=0.0 velocity=0.0; origin xyz=-0.05299  0.00815 -0.09666 rpy=0  0  0 -> xyz=0.06298  0.00427 -0.09073 rpy=0 0 0
- joint hand_left_index_joint1: axis 0.99581  0.05254  0.07483 -> -4.5000e-04 -7.8515e-01  6.1929e-01; limit lower=0.0 upper=0.0 effort=0.0 velocity=0.0 -> lower=-3.14159265359 upper=3.14159265359 effort=0.0 velocity=0.0; origin xyz=0.00336 -0.00083 -0.04486 rpy=0  0  0 -> xyz=0.0255  -0.02293 -0.02913 rpy=0 0 0
- joint hand_left_index_joint2: axis 0.99581  0.05254  0.07483 -> -4.5000e-04 -7.8515e-01  6.1929e-01; limit lower=0.0 upper=0.0 effort=0.0 velocity=0.0 -> lower=-3.14159265359 upper=3.14159265359 effort=0.0 velocity=0.0; origin xyz=0.00192 -0.00048 -0.02592 rpy=0  0  0 -> xyz=0.01473 -0.01323 -0.01684 rpy=0 0 0
- joint hand_left_little_joint0: axis -0.99581 -0.05254 -0.07483 -> 4.5000e-04  7.8515e-01 -6.1929e-01; limit lower=0.0 upper=0.0 effort=0.0 velocity=0.0 -> lower=-3.14159265359 upper=3.14159265359 effort=0.0 velocity=0.0; origin xyz=0.02535  0.01177 -0.11388 rpy=0  0  0 -> xyz=0.076   -0.06788 -0.05801 rpy=0 0 0
- joint hand_left_little_joint1: axis 0.98736  0.04706 -0.15134 -> 0.12702 -0.87986  0.45793; limit lower=0.0 upper=0.0 effort=0.0 velocity=0.0 -> lower=-3.14159265359 upper=3.14159265359 effort=0.0 velocity=0.0; origin xyz=-4.78000000e-03  -1.00000000e-05  -2.55800000e-02 rpy=0  0  0 -> xyz=0.0149  -0.00731 -0.02003 rpy=0 0 0
- joint hand_left_little_joint2: axis 0.98736  0.04706 -0.15134 -> 0.12702 -0.87986  0.45793; limit lower=0.0 upper=0.0 effort=0.0 velocity=0.0 -> lower=-3.14159265359 upper=3.14159265359 effort=0.0 velocity=0.0; origin xyz=-0.00395 -0.00077 -0.02568 rpy=0  0  0 -> xyz=0.01435 -0.00829 -0.02003 rpy=0 0 0
- joint hand_left_middle_joint0: axis -0.99386 -0.04855  0.09942 -> -0.09794  0.86187 -0.49757; limit lower=0.0 upper=0.0 effort=0.0 velocity=0.0 -> lower=-3.14159265359 upper=3.14159265359 effort=0.0 velocity=0.0; origin xyz=-0.02964  0.00901 -0.11157 rpy=0  0  0 -> xyz=0.07239 -0.02163 -0.08775 rpy=0 0 0
- joint hand_left_middle_joint1: axis 0.99386  0.04855 -0.09942 -> 0.09794 -0.86187  0.49757; limit lower=0.0 upper=0.0 effort=0.0 velocity=0.0 -> lower=-3.14159265359 upper=3.14159265359 effort=0.0 velocity=0.0; origin xyz=-0.00446 -0.00122 -0.04476 rpy=0  0  0 -> xyz=0.02511 -0.01644 -0.03352 rpy=0 0 0
- joint hand_left_middle_joint2: axis 0.99386  0.04855 -0.09942 -> 0.09794 -0.86187  0.49757; limit lower=0.0 upper=0.0 effort=0.0 velocity=0.0 -> lower=-3.14159265359 upper=3.14159265359 effort=0.0 velocity=0.0; origin xyz=-0.0026  -0.00071 -0.02586 rpy=0  0  0 -> xyz=0.0145  -0.00948 -0.01938 rpy=0 0 0
- joint hand_left_ring_joint0: axis 0.99863  0.05074 -0.01234 -> 0.04893 -0.82665  0.56057; limit lower=0.0 upper=0.0 effort=0.0 velocity=0.0 -> lower=-3.14159265359 upper=3.14159265359 effort=0.0 velocity=0.0; origin xyz=-0.00289  0.01018 -0.12037 rpy=0  0  0 -> xyz=0.07849 -0.04758 -0.0786 rpy=0 0 0
- joint hand_left_ring_joint1: axis 0.99863  0.05074 -0.01234 -> 0.04893 -0.82665  0.56057; limit lower=0.0 upper=0.0 effort=0.0 velocity=0.0 -> lower=-3.14159265359 upper=3.14159265359 effort=0.0 velocity=0.0; origin xyz=-0.00055 -0.00103 -0.04498 rpy=0  0  0 -> xyz=0.0254  -0.01976 -0.03145 rpy=0 0 0
- joint hand_left_ring_joint2: axis 0.99863  0.05074 -0.01234 -> 0.04893 -0.82665  0.56057; limit lower=0.0 upper=0.0 effort=0.0 velocity=0.0 -> lower=-3.14159265359 upper=3.14159265359 effort=0.0 velocity=0.0; origin xyz=-0.00034 -0.00059 -0.02599 rpy=0  0  0 -> xyz=0.01467 -0.0114  -0.01818 rpy=0 0 0
- joint hand_left_thumb_joint0: axis 0.01118  0.0229   0.99967 -> -0.56454  0.4401   0.69828; limit lower=0.0 upper=0.0 effort=0.0 velocity=0.0 -> lower=-3.14159265359 upper=3.14159265359 effort=0.0 velocity=0.0; origin xyz=0.02063 -0.00513 -0.05274 rpy=0  0  0 -> xyz=0.02661 -0.04226 -0.02719 rpy=0 0 0
- joint hand_left_thumb_joint1: axis -0.05101  0.99844 -0.02231 -> 0.82395 0.35063 0.44515; limit lower=0.0 upper=0.0 effort=0.0 velocity=0.0 -> lower=-3.14159265359 upper=3.14159265359 effort=0.0 velocity=0.0; origin xyz=0.04388 -0.00276 -0.009 rpy=0  0  0 -> xyz=0.00302 -0.04166  0.01642 rpy=0 0 0
- joint hand_left_thumb_joint2: axis 0.05101 -0.99844  0.02231 -> -0.82395 -0.35063 -0.44515; limit lower=0.0 upper=0.0 effort=0.0 velocity=0.0 -> lower=-3.14159265359 upper=3.14159265359 effort=0.0 velocity=0.0; origin xyz=0.02596  0.00126 -0.00032 rpy=0  0  0 -> xyz=0.00123 -0.02151  0.01455 rpy=0 0 0
- joint hand_right_index_joint0: axis 0.99272 -0.10801 -0.0532 -> -4.5000e-04  7.8515e-01 -6.1929e-01; limit lower=0.0 upper=0.0 effort=0.0 velocity=0.0 -> lower=-3.14159265359 upper=3.14159265359 effort=0.0 velocity=0.0; origin xyz=-0.03947 -0.06578 -0.09727 rpy=0  0  0 -> xyz=-0.07882 -0.07793 -0.05531 rpy=0 0 0
- joint hand_right_index_joint1: axis 0.99272 -0.10801 -0.0532 -> -4.5000e-04  7.8515e-01 -6.1929e-01; limit lower=0.0 upper=0.0 effort=0.0 velocity=0.0 -> lower=-3.14159265359 upper=3.14159265359 effort=0.0 velocity=0.0; origin xyz=-0.00485 -0.02937 -0.03374 rpy=0  0  0 -> xyz=-0.0255  -0.02285 -0.02919 rpy=0 0 0
- joint hand_right_index_joint2: axis 0.99272 -0.10801 -0.0532 -> -4.5000e-04  7.8515e-01 -6.1929e-01; limit lower=0.0 upper=0.0 effort=0.0 velocity=0.0 -> lower=-3.14159265359 upper=3.14159265359 effort=0.0 velocity=0.0; origin xyz=-0.00294 -0.01695 -0.01948 rpy=0  0  0 -> xyz=-0.01473 -0.01331 -0.01678 rpy=0 0 0
- joint hand_right_little_joint0: axis 0.99228  0.04151  0.1168 -> 0.12702  0.87986 -0.45793; limit lower=0.0 upper=0.0 effort=0.0 velocity=0.0 -> lower=-3.14159265359 upper=3.14159265359 effort=0.0 velocity=0.0; origin xyz=0.03945 -0.06054 -0.08578 rpy=0  0  0 -> xyz=-0.06707 -0.00672 -0.08965 rpy=0 0 0
- joint hand_right_little_joint1: axis 0.99228  0.04151  0.1168 -> 0.12702  0.87986 -0.45793; limit lower=0.0 upper=0.0 effort=0.0 velocity=0.0 -> lower=-3.14159265359 upper=3.14159265359 effort=0.0 velocity=0.0; origin xyz=0.00313 -0.01715 -0.01928 rpy=0  0  0 -> xyz=-0.01433 -0.0082  -0.02007 rpy=0 0 0
- joint hand_right_little_joint2: axis 0.99228  0.04151  0.1168 -> 0.12702  0.87986 -0.45793; limit lower=0.0 upper=0.0 effort=0.0 velocity=0.0 -> lower=-3.14159265359 upper=3.14159265359 effort=0.0 velocity=0.0; origin xyz=0.00294 -0.01716 -0.0193 rpy=0  0  0 -> xyz=-0.01436 -0.00838 -0.01998 rpy=0 0 0
- joint hand_right_middle_joint0: axis 0.99863 -0.05074  0.01234 -> 0.04893  0.82665 -0.56057; limit lower=0.0 upper=0.0 effort=0.0 velocity=0.0 -> lower=-3.14159265359 upper=3.14159265359 effort=0.0 velocity=0.0; origin xyz=-0.01152 -0.07229 -0.10272 rpy=0  0  0 -> xyz=-0.0818  -0.05804 -0.07648 rpy=0 0 0
- joint hand_right_middle_joint1: axis 0.99863 -0.05074  0.01234 -> 0.04893  0.82665 -0.56057; limit lower=0.0 upper=0.0 effort=0.0 velocity=0.0 -> lower=-3.14159265359 upper=3.14159265359 effort=0.0 velocity=0.0; origin xyz=-0.00094 -0.02967 -0.03381 rpy=0  0  0 -> xyz=-0.02539 -0.01968 -0.0315 rpy=0 0 0
- joint hand_right_middle_joint2: axis 0.99863 -0.05074  0.01234 -> 0.04893  0.82665 -0.56057; limit lower=0.0 upper=0.0 effort=0.0 velocity=0.0 -> lower=-3.14159265359 upper=3.14159265359 effort=0.0 velocity=0.0; origin xyz=-0.00068 -0.01714 -0.01953 rpy=0  0  0 -> xyz=-0.01468 -0.01148 -0.01812 rpy=0 0 0
- joint hand_right_ring_joint0: axis 0.99694  0.00691  0.07778 -> 0.09794  0.86187 -0.49757; limit lower=0.0 upper=0.0 effort=0.0 velocity=0.0 -> lower=-3.14159265359 upper=3.14159265359 effort=0.0 velocity=0.0; origin xyz=0.01553 -0.06864 -0.09667 rpy=0  0  0 -> xyz=-0.07619 -0.03244 -0.08626 rpy=0 0 0
- joint hand_right_ring_joint1: axis 0.99694  0.00691  0.07778 -> 0.09794  0.86187 -0.49757; limit lower=0.0 upper=0.0 effort=0.0 velocity=0.0 -> lower=-3.14159265359 upper=3.14159265359 effort=0.0 velocity=0.0; origin xyz=0.00298 -0.02975 -0.03362 rpy=0  0  0 -> xyz=-0.0251  -0.01635 -0.03357 rpy=0 0 0
- joint hand_right_ring_joint2: axis 0.99694  0.00691  0.07778 -> 0.09794  0.86187 -0.49757; limit lower=0.0 upper=0.0 effort=0.0 velocity=0.0 -> lower=-3.14159265359 upper=3.14159265359 effort=0.0 velocity=0.0; origin xyz=0.00158 -0.01719 -0.01943 rpy=0  0  0 -> xyz=-0.01451 -0.00956 -0.01933 rpy=0 0 0
- joint hand_right_thumb_joint0: axis 0.02421  0.65934  0.75145 -> 0.56454 0.4401  0.69828; limit lower=0.0 upper=0.0 effort=0.0 velocity=0.0 -> lower=-3.14159265359 upper=3.14159265359 effort=0.0 velocity=0.0; origin xyz=-0.02237 -0.03474 -0.03349 rpy=0  0  0 -> xyz=-0.02435 -0.0405  -0.0244 rpy=0 0 0
- joint hand_right_thumb_joint1: axis -0.04626 -0.75013  0.65966 -> 0.82395 -0.35063 -0.44515; limit lower=0.0 upper=0.0 effort=0.0 velocity=0.0 -> lower=-3.14159265359 upper=3.14159265359 effort=0.0 velocity=0.0; origin xyz=-0.04393 -0.00576 -0.01691 rpy=0  0  0 -> xyz=-0.01601 -0.04225  0.01441 rpy=0 0 0
- joint hand_right_thumb_joint2: axis 0.04626  0.75013 -0.65966 -> -0.82395  0.35063  0.44515; limit lower=0.0 upper=0.0 effort=0.0 velocity=0.0 -> lower=-3.14159265359 upper=3.14159265359 effort=0.0 velocity=0.0; origin xyz=-0.02596  0.00135 -0.00035 rpy=0  0  0 -> xyz=-0.00131 -0.02147  0.01459 rpy=0 0 0
- joint neck_axis0: origin xyz=0       0.00152  0.71567 rpy=0  0  0 -> xyz=0      0.00152 0.71067 rpy=0 0 0
- joint neck_axis1: origin xyz=0  0  0 rpy=0  0  0 -> xyz=0 0 0 rpy=0 0 0
- joint neck_axis2: axis 0  0  1 -> 0 0 1; origin xyz=0  0  0 rpy=0  0  0 -> xyz=0 0 0 rpy=0 0 0
- joint shoulder_left_axis0: axis 1 0 0 -> 0.82395 0.35063 0.44515; origin xyz=0.29189  0.01393  0.54489 rpy=0  0  0 -> xyz=0.29189 0.01393 0.54489 rpy=0 0 0
- joint shoulder_left_axis1: axis 0 1 0 -> 0.04893 -0.82665  0.56057; origin xyz=0  0  0 rpy=0  0  0 -> xyz=0 0 0 rpy=0 0 0
- joint shoulder_left_axis2: axis 1 0 0 -> 0.56454 -0.4401  -0.69828; origin xyz=0  0  0 rpy=0  0  0 -> xyz=0 0 0 rpy=0 0 0
- joint shoulder_right_axis0: axis 1 0 0 -> -0.82395  0.35063  0.44515; origin xyz=-0.29317  0.00923  0.5481 rpy=0  0  0 -> xyz=-0.29306  0.01109  0.54684 rpy=0 0 0
- joint shoulder_right_axis1: axis 0 1 0 -> 0.04893  0.82665 -0.56057; origin xyz=0  0  0 rpy=0  0  0 -> xyz=0 0 0 rpy=0 0 0
- joint shoulder_right_axis2: axis 1 0 0 -> -0.56454 -0.4401  -0.69828; origin xyz=0  0  0 rpy=0  0  0 -> xyz=0 0 0 rpy=0 0 0
- joint wrist_left_axis0: axis -0.05101  0.99844 -0.02231 -> 0.82395 0.35063 0.44515; origin xyz=-0.01364 -0.00601 -0.23778 rpy=0  0  0 -> xyz=0.13382 -0.09565 -0.17235 rpy=0 0 0
- joint wrist_left_axis1: axis 0.99863  0.05074 -0.01234 -> 0.04893 -0.82665  0.56057; origin xyz=0  0  0 rpy=0  0  0 -> xyz=0 0 0 rpy=0 0 0
- joint wrist_left_axis2: axis -0.01118 -0.0229  -0.99967 -> 0.56454 -0.4401  -0.69828; origin xyz=0  0  0 rpy=0  0  0 -> xyz=0 0 0 rpy=0 0 0
- joint wrist_right_axis0: axis 0.99863 -0.05074  0.01234 -> 0.04893  0.82665 -0.56057; origin xyz=0.00534 -0.15418 -0.17495 rpy=0  0  0 -> xyz=-0.131   -0.09345 -0.16886 rpy=0 0 0
- joint wrist_right_axis1: axis -0.04626 -0.75013  0.65966 -> 0.82395 -0.35063 -0.44515; origin xyz=0  0  0 rpy=0  0  0 -> xyz=0 0 0 rpy=0 0 0
- joint wrist_right_axis2: axis -0.02421 -0.65934 -0.75145 -> -0.56454 -0.4401  -0.69828; origin xyz=0  0  0 rpy=0  0  0 -> xyz=0 0 0 rpy=0 0 0

Commit message: Remove zed cam

File: roboy_icecream/model.urdf (robot description, URDF)
Before this commit: robot roboy_icecream, 63 links, 62 joints
Links:
- removed link zed_camera
- removed link zed_camera_left_lense
- removed link zed_camera_right_lense
Joints:
- removed joint zed_camera_left
- removed joint zed_camera_mount
- removed joint zed_camera_right

Commit message: Fix joints of foot_tips

File: roboy_icecream/model.urdf (robot description, URDF)
Before this commit: robot roboy_icecream, 60 links, 59 joints
Joints:
- joint joint_foot_left_tip: axis 0  0  0 -> 0  0  1
- joint joint_foot_right_tip: axis 0  0  0 -> 0  0  1

Commit message: works with trackers

File: roboy_icecream/model.urdf (robot description, URDF)
Before this commit: robot roboy_icecream, 25 links, 24 joints
Joints:
- joint shoulder_left_axis0: axis -0.99863 -0.05074  0.01234 -> 1 0 0
- joint shoulder_left_axis1: axis -0.05101  0.99844 -0.02231 -> 0 1 0
- joint shoulder_left_axis2: axis -0.01118 -0.0229  -0.99967 -> 0 0 1
- joint shoulder_right_axis0: axis 0.99863 -0.05074  0.01234 -> 1 0 0
- joint shoulder_right_axis1: axis -0.05101 -0.99844  0.02231 -> 0 1 0
- joint shoulder_right_axis2: axis 0.01118 -0.0229  -0.99967 -> 0 0 1
