Commit message: Add virtual ball joint in scooper

File: roboy_icecream/model.urdf (robot description, URDF)
Before this commit: robot roboy_icecream, 52 links, 51 joints
Links:
- added link scooper_dummy_axis0, mass 0
- added link scooper_dummy_axis1, mass 0
- added link scooper_dummy_axis2, mass 0
Joints:
- added joint scooper_dummy_joint0: type continuous, parent scooper, child scooper_dummy_axis0, origin xyz=0.04902 -0.12131  0.00304 rpy=0 0 0, axis 1 0 0, limit lower=0 upper=0 effort=0 velocity=0
- added joint scooper_dummy_joint1: type continuous, parent scooper_dummy_axis0, child scooper_dummy_axis1, origin xyz=0 0 0 rpy=0 0 0, axis 0 1 0, limit lower=0 upper=0 effort=0 velocity=0
- added joint scooper_dummy_joint2: type continuous, parent scooper_dummy_axis1, child scooper_dummy_axis2, origin xyz=0 0 0 rpy=0 0 0, axis 0 0 1, limit lower=0 upper=0 effort=0 velocity=0
- joint scooper_palm: limit lower=3.14 upper=3.14 effort=0.0 velocity=0.0 -> lower=0 upper=0 effort=0.0 velocity=0.0; origin xyz=-0.01686  0.00755 -0.06248 rpy=0 0 0 -> xyz=-0.01686  0.00755 -0.06248 rpy=3.14 0 0; type revolute -> fixed
- joint shoulder_right_axis0: axis 0.99863 -0.05074  0.01234 -> 1 0 0; limit lower=-1.57 upper=0.0 effort=0.0 velocity=0.0 -> lower=-1.87 upper=0.88 effort=0.0 velocity=0.0
- joint shoulder_right_axis1: axis -0.05101 -0.99844  0.02231 -> 0 1 0; limit lower=0.0 upper=1.57 effort=0.0 velocity=0.0 -> lower=-0.2 upper=1.463 effort=0.0 velocity=0.0
- joint shoulder_right_axis2: axis 0.01118 -0.0229  -0.99967 -> 0 0 1

Commit message: Set joint limits for left shoulder

File: roboy_icecream/model.urdf (robot description, URDF)
Before this commit: robot roboy_icecream, 55 links, 54 joints
Joints:
- joint shoulder_left_axis0: limit lower=-3.14159265359 upper=3.14159265359 effort=0.0 velocity=0.0 -> lower=-1.87 upper=0.88 effort=0.0 velocity=0.0
- joint shoulder_left_axis1: limit lower=-3.14159265359 upper=3.14159265359 effort=0.0 velocity=0.0 -> lower=-0.2 upper=1.463 effort=0.0 velocity=0.0
- joint shoulder_left_axis2: limit lower=-3.14159265359 upper=3.14159265359 effort=0.0 velocity=0.0 -> lower=-0.6 upper=0.6 effort=0.0 velocity=0.0
- joint shoulder_right_axis2: limit lower=-1.57 upper=1.57 effort=0.0 velocity=0.0 -> lower=-0.6 upper=0.6 effort=0.0 velocity=0.0

Commit message: Fix model to be cardsflow compatible

File: roboy_icecream/model.urdf (robot description, URDF)
Before this commit: robot roboy_icecream, 55 links, 54 joints
Joints:
- joint hand_left_index_joint0: type fixed -> revolute
- joint hand_left_index_joint1: type fixed -> revolute
- joint hand_left_index_joint2: type fixed -> revolute
- joint hand_left_little_joint0: type fixed -> revolute
- joint hand_left_little_joint1: type fixed -> revolute
- joint hand_left_little_joint2: type fixed -> revolute
- joint hand_left_middle_joint0: type fixed -> revolute
- joint hand_left_middle_joint1: type fixed -> revolute
- joint hand_left_middle_joint2: type fixed -> revolute
- joint hand_left_ring_joint0: type fixed -> revolute
- joint hand_left_ring_joint1: type fixed -> revolute
- joint hand_left_ring_joint2: type fixed -> revolute
- joint hand_left_thumb_joint0: type fixed -> revolute
- joint hand_left_thumb_joint1: type fixed -> revolute
- joint hand_left_thumb_joint2: type fixed -> revolute
- joint hand_right_index_joint0: type fixed -> revolute
- joint hand_right_index_joint1: type fixed -> revolute
- joint hand_right_index_joint2: type fixed -> revolute
- joint hand_right_little_joint0: type fixed -> revolute
- joint hand_right_little_joint1: type fixed -> revolute
- joint hand_right_little_joint2: type fixed -> revolute
- joint hand_right_middle_joint0: type fixed -> revolute
- joint hand_right_middle_joint1: type fixed -> revolute
- joint hand_right_middle_joint2: type fixed -> revolute
- joint hand_right_ring_joint0: type fixed -> revolute
- joint hand_right_ring_joint1: type fixed -> revolute
- joint hand_right_ring_joint2: type fixed -> revolute
- joint hand_right_thumb_joint0: type fixed -> revolute
- joint hand_right_thumb_joint1: type fixed -> revolute
- joint hand_right_thumb_joint2: type fixed -> revolute
- joint scooper_dummy_joint0: limit lower=0 upper=0 effort=0 velocity=0 -> lower=-3.14 upper=3.14 effort=0 velocity=0; type continuous -> revolute
- joint scooper_dummy_joint1: limit lower=0 upper=0 effort=0 velocity=0 -> lower=-3.14 upper=3.14 effort=0 velocity=0; type continuous -> revolute
- joint scooper_dummy_joint2: limit lower=0 upper=0 effort=0 velocity=0 -> lower=-3.14 upper=3.14 effort=0 velocity=0; type continuous -> revolute
- joint scooper_palm: type fixed -> revolute
- joint spine: type fixed -> revolute
- joint zed_camera_left: type fixed -> revolute
- joint zed_camera_mount: type fixed -> revolute
- joint zed_camera_right: type fixed -> revolute

Commit message: Fix the ice cream box stl files

File: roboy_icecream/model.urdf (robot description, URDF)
Before this commit: robot roboy_icecream, 55 links, 54 joints
Joints:
- joint hand_left_index_joint0: type revolute -> fixed
- joint hand_left_index_joint1: type revolute -> fixed
- joint hand_left_index_joint2: type revolute -> fixed
- joint hand_left_little_joint0: type revolute -> fixed
- joint hand_left_little_joint1: type revolute -> fixed
- joint hand_left_little_joint2: type revolute -> fixed
- joint hand_left_middle_joint0: type revolute -> fixed
- joint hand_left_middle_joint1: type revolute -> fixed
- joint hand_left_middle_joint2: type revolute -> fixed
- joint hand_left_ring_joint0: type revolute -> fixed
- joint hand_left_ring_joint1: type revolute -> fixed
- joint hand_left_ring_joint2: type revolute -> fixed
- joint hand_left_thumb_joint0: type revolute -> fixed
- joint hand_left_thumb_joint1: type revolute -> fixed
- joint hand_left_thumb_joint2: type revolute -> fixed
- joint hand_right_index_joint0: type revolute -> fixed
- joint hand_right_index_joint1: type revolute -> fixed
- joint hand_right_index_joint2: type revolute -> fixed
- joint hand_right_little_joint0: type revolute -> fixed
- joint hand_right_little_joint1: type revolute -> fixed
- joint hand_right_little_joint2: type revolute -> fixed
- joint hand_right_middle_joint0: type revolute -> fixed
- joint hand_right_middle_joint1: type revolute -> fixed
- joint hand_right_middle_joint2: type revolute -> fixed
- joint hand_right_ring_joint0: type revolute -> fixed
- joint hand_right_ring_joint1: type revolute -> fixed
- joint hand_right_ring_joint2: type revolute -> fixed
- joint hand_right_thumb_joint0: type revolute -> fixed
- joint hand_right_thumb_joint1: type revolute -> fixed
- joint hand_right_thumb_joint2: type revolute -> fixed
- joint ice_left_linear: limit lower=0.0 upper=0.0 effort=0.0 velocity=0.0 -> lower=0.25 upper=0.25 effort=0.0 velocity=0.0
- joint ice_right_linear: limit lower=0.0 upper=0.0 effort=0.0 velocity=0.0 -> lower=0.25 upper=0.25 effort=0.0 velocity=0.0
- joint scooper_dummy_joint0: limit lower=-3.14 upper=3.14 effort=0 velocity=0 -> lower=0 upper=0 effort=0 velocity=0; type revolute -> continuous
- joint scooper_dummy_joint1: limit lower=-3.14 upper=3.14 effort=0 velocity=0 -> lower=0 upper=0 effort=0 velocity=0; type revolute -> continuous
- joint scooper_dummy_joint2: limit lower=-3.14 upper=3.14 effort=0 velocity=0 -> lower=0 upper=0 effort=0 velocity=0; type revolute -> continuous
- joint scooper_palm: type revolute -> fixed
- joint spine: type revolute -> fixed
- joint zed_camera_left: type revolute -> fixed
- joint zed_camera_mount: type revolute -> fixed
- joint zed_camera_right: type revolute -> fixed

Commit message: Change axes in moveIT urdf model

File: roboy_icecream/model.urdf (robot description, URDF)
Before this commit: robot roboy_icecream, 55 links, 54 joints
Joints:
- joint shoulder_right_axis0: axis 1 0 0 -> 0.99863 -0.05074  0.01234; limit lower=-1.87 upper=0.88 effort=0.0 velocity=0.0 -> lower=-3.14 upper=3.14 effort=0.0 velocity=0.0
- joint shoulder_right_axis1: axis 0 1 0 -> -0.05101 -0.99844  0.02231; limit lower=-0.2 upper=1.463 effort=0.0 velocity=0.0 -> lower=-3.14 upper=3.14 effort=0.0 velocity=0.0
- joint shoulder_right_axis2: axis 0 0 1 -> 0.01118 -0.0229  -0.99967; limit lower=-0.6 upper=0.6 effort=0.0 velocity=0.0 -> lower=-3.14 upper=3.14 effort=0.0 velocity=0.0

Commit message: Set axes for previously fixed joints

File: roboy_icecream/model.urdf (robot description, URDF)
Before this commit: robot roboy_icecream, 56 links, 55 joints
Joints:
- joint zed_camera_left: axis 0 0 0 -> 1 0 0
- joint zed_camera_mount: axis 0 0 0 -> 1 0 0
- joint zed_camera_right: axis 0 0 0 -> 1 0 0
- joint zed_mini_attachement: axis 0 0 0 -> 1 0 0
- joint zed_pico_attachement: axis 0 0 0 -> 1 0 0

Commit message: Move ball joint to the scooper ball

File: roboy_icecream/model.urdf (robot description, URDF)
Before this commit: robot roboy_icecream, 56 links, 55 joints
Joints:
- joint scooper_axis0: axis 5.0740e-02 9.9871e-01 3.7000e-04 -> 0 1 0; child sphere_link1 -> scooper
- joint scooper_axis1: axis -0.99863  0.05074 -0.01234 -> -1 0 0; child sphere_link2 -> sphere_link1; origin xyz=0 0 0 rpy=0 0 0 -> xyz=0 -0.085 0 rpy=0 0 0; parent sphere_link1 -> scooper
- joint scooper_axis2: child scooper -> sphere_link2; parent sphere_link2 -> sphere_link1

Commit message: Add reduced meshes for moveIT

File: roboy_icecream/model.urdf (robot description, URDF)
Before this commit: robot roboy_icecream, 56 links, 55 joints
Links:
- added link sphere_link3, mass 0.002996372533076606
- link sphere_link1: geometry 
- link sphere_link2: geometry 
Joints:
- added joint scooper_axis3: type revolute, parent sphere_link2, child sphere_link3, origin xyz=0 0 0 rpy=0 0 0, axis 0 0 1, limit lower=-3.14159265359 upper=3.14159265359 effort=0.0 velocity=0.0
- joint scooper_axis2: axis -1.2340e-02  2.5000e-04  9.9992e-01 -> 0 -1 0

Commit message: dont move scooper palm

File: roboy_icecream/model.urdf (robot description, URDF)
Before this commit: robot roboy_icecream, 57 links, 56 joints
Joints:
- joint palm_scooper: limit lower=-1.57079632679 upper=1.57079632679 effort=0.0 velocity=0.0 -> lower=0.0 upper=0.0 effort=0.0 velocity=0.0

Commit message: axis

File: roboy_icecream/model.urdf (robot description, URDF)
Before this commit: robot roboy_icecream, 57 links, 56 joints
Joints:
- joint shoulder_right_axis0: axis 0.99863 -0.05074  0.01234 -> 1 0 0
- joint shoulder_right_axis1: axis -5.07400000e-02  -9.98710000e-01  -3.70000000e-04 -> 0 1 0
- joint shoulder_right_axis2: axis 1.23400000e-02  -2.50000000e-04  -9.99920000e-01 -> 0 0 1

Commit message: Adapt limits

File: roboy_icecream/model.urdf (robot description, URDF)
Before this commit: robot roboy_icecream, 57 links, 56 joints
Joints:
- joint elbow_right: limit lower=0.0 upper=1.91986217719 effort=0.0 velocity=0.0 -> lower=0.0 upper=10 effort=0.0 velocity=0.0
- joint wrist_right: limit lower=-0.872664625997 upper=0.872664625997 effort=0.0 velocity=0.0 -> lower=-180 upper=180 effort=0.0 velocity=0.0

Commit message: Reintroduce cardsflow.urdf

File: roboy_icecream/model.urdf (robot description, URDF)
Before this commit: robot roboy_icecream, 57 links, 56 joints
Joints:
- joint elbow_right: limit lower=0.0 upper=10 effort=0.0 velocity=0.0 -> lower=0.0 upper=1.91986217719 effort=0.0 velocity=0.0
- joint palm_scooper: limit lower=0.0 upper=0.0 effort=0.0 velocity=0.0 -> lower=-1.57079632679 upper=1.57079632679 effort=0.0 velocity=0.0
- joint shoulder_right_axis0: axis 1 0 0 -> 0.99863 -0.05074  0.01234
- joint shoulder_right_axis1: axis 0 1 0 -> -5.07400000e-02  -9.98710000e-01  -3.70000000e-04
- joint shoulder_right_axis2: axis 0 0 1 -> 1.23400000e-02  -2.50000000e-04  -9.99920000e-01
- joint wrist_right: limit lower=-180 upper=180 effort=0.0 velocity=0.0 -> lower=-0.872664625997 upper=0.872664625997 effort=0.0 velocity=0.0

Commit message: Set scooper_palm to fixed

File: roboy_icecream/model.urdf (robot description, URDF)
Before this commit: robot roboy_icecream, 57 links, 56 joints
Joints:
- joint palm_scooper: type revolute -> fixed

Commit message: Remove hands for moveit planning

File: roboy_icecream/model.urdf (robot description, URDF)
Before this commit: robot roboy_icecream, 57 links, 56 joints
Links:
- removed link hand_left_index_link0
- removed link hand_left_index_link1
- removed link hand_left_index_link2
- removed link hand_left_little_link0
- removed link hand_left_little_link1
- removed link hand_left_little_link2
- removed link hand_left_middle_link0
- removed link hand_left_middle_link1
- removed link hand_left_middle_link2
- removed link hand_left_ring_link0
- removed link hand_left_ring_link1
- removed link hand_left_ring_link2
- removed link hand_left_thumb_link0
- removed link hand_left_thumb_link1
- removed link hand_left_thumb_link2
- removed link hand_right_index_link0
- removed link hand_right_index_link1
- removed link hand_right_index_link2
- removed link hand_right_little_link0
- removed link hand_right_little_link1
- removed link hand_right_little_link2
- removed link hand_right_middle_link0
- removed link hand_right_middle_link1
- removed link hand_right_middle_link2
- removed link hand_right_ring_link0
- removed link hand_right_ring_link1
- removed link hand_right_ring_link2
- removed link hand_right_thumb_link0
- removed link hand_right_thumb_link1
- removed link hand_right_thumb_link2
Joints:
- removed joint hand_left_index_joint0
- removed joint hand_left_index_joint1
- removed joint hand_left_index_joint2
- removed joint hand_left_little_joint0
- removed joint hand_left_little_joint1
- removed joint hand_left_little_joint2
- removed joint hand_left_middle_joint0
- removed joint hand_left_middle_joint1
- removed joint hand_left_middle_joint2
- removed joint hand_left_ring_joint0
- removed joint hand_left_ring_joint1
- removed joint hand_left_ring_joint2
- removed joint hand_left_thumb_joint0
- removed joint hand_left_thumb_joint1
- removed joint hand_left_thumb_joint2
- removed joint hand_right_index_joint0
- removed joint hand_right_index_joint1
- removed joint hand_right_index_joint2
- removed joint hand_right_little_joint0
- removed joint hand_right_little_joint1
- removed joint hand_right_little_joint2
- removed joint hand_right_middle_joint0
- removed joint hand_right_middle_joint1
- removed joint hand_right_middle_joint2
- removed joint hand_right_ring_joint0
- removed joint hand_right_ring_joint1
- removed joint hand_right_ring_joint2
- removed joint hand_right_thumb_joint0
- removed joint hand_right_thumb_joint1
- removed joint hand_right_thumb_joint2

Commit message: Remove camera stuff

File: roboy_icecream/model.urdf (robot description, URDF)
Before this commit: robot roboy_icecream, 27 links, 26 joints
Links:
- removed link pico_flexx
- removed link zed_camera
- removed link zed_camera_left_lense
- removed link zed_camera_right_lense
- removed link zed_mini
Joints:
- removed joint zed_camera_left
- removed joint zed_camera_mount
- removed joint zed_camera_right
- removed joint zed_mini_attachement
- removed joint zed_pico_attachement

Commit message: Joint limits

File: roboy_icecream/model.urdf (robot description, URDF)
Before this commit: robot roboy_icecream, 22 links, 21 joints
Joints:
- joint shoulder_right_axis0: axis 0.99863 -0.05074  0.01234 -> 1 0 0; limit lower=-3.14159265359 upper=3.14159265359 effort=0.0 velocity=0.0 -> lower=-1.57 upper=1.57 effort=0.0 velocity=0.0
- joint shoulder_right_axis1: axis -5.07400000e-02  -9.98710000e-01  -3.70000000e-04 -> 0 1 0; limit lower=-3.14159265359 upper=3.14159265359 effort=0.0 velocity=0.0 -> lower=-0.2 upper=1.57 effort=0.0 velocity=0.0
- joint shoulder_right_axis2: axis 1.23400000e-02  -2.50000000e-04  -9.99920000e-01 -> 0 0 1
- joint wrist_right: limit lower=-0.872664625997 upper=0.872664625997 effort=0.0 velocity=0.0 -> lower=-2 upper=2 effort=0.0 velocity=0.0

Commit message: with correct axis for shoulder right

File: roboy_icecream/model.urdf (robot description, URDF)
Before this commit: robot roboy_icecream, 57 links, 56 joints
Joints:
- joint shoulder_left_axis0: axis -0.99863 -0.05074  0.01234 -> 1 0 0
- joint shoulder_left_axis1: axis -0.05101  0.99844 -0.02231 -> 0 1 0
- joint shoulder_left_axis2: axis -0.01118 -0.0229  -0.99967 -> 0 0 1

Commit message: Dunno what I'm doin

File: roboy_icecream/model.urdf (robot description, URDF)
Before this commit: robot roboy_icecream, 22 links, 21 joints
Joints:
- joint elbow_right: limit lower=0.0 upper=1.91986217719 effort=0.0 velocity=0.0 -> lower=0.0 upper=2.1 effort=0.0 velocity=0.0
- joint shoulder_right_axis2: limit lower=-3.14159265359 upper=3.14159265359 effort=0.0 velocity=0.0 -> lower=-0.3 upper=2.2 effort=0.0 velocity=0.0

Commit message: joint limits and minor stuff?

File: roboy_icecream/model.urdf (robot description, URDF)
Before this commit: robot roboy_icecream, 20 links, 19 joints
Joints:
- joint wrist_right: limit lower=-2 upper=2 effort=0.0 velocity=0.0 -> lower=-3.14 upper=3.14 effort=0.0 velocity=0.0

Commit message: da best

File: roboy_icecream/model.urdf (robot description, URDF)
Before this commit: robot roboy_icecream, 19 links, 18 joints
Joints:
- joint elbow_left: type fixed -> revolute
- joint shoulder_left_axis0: axis -0.99863 -0.05074  0.01234 -> 1 0 0
- joint shoulder_left_axis1: axis -0.05101  0.99844 -0.02231 -> 0 1 0
- joint shoulder_left_axis2: axis -0.01118 -0.0229  -0.99967 -> 0 0 1
- joint shoulder_right_axis0: axis 0.99863 -0.05074  0.01234 -> 1 0 0
- joint shoulder_right_axis1: axis -5.0740e-02 -9.9871e-01 -3.7000e-04 -> 0 1 0
- joint shoulder_right_axis2: axis 1.2340e-02 -2.5000e-04 -9.9992e-01 -> 0 0 1
- joint spine: type fixed -> revolute
- joint zed_camera_left: type fixed -> revolute
- joint zed_camera_mount: type fixed -> revolute
- joint zed_camera_right: type fixed -> revolute
- joint zed_mini_attachement: type fixed -> revolute
- joint zed_pico_attachement: type fixed -> revolute
